File: Hardware/Kicad/Routing/ProjetSNES2023ENSEA.kicad_pcb (KiCad board)
At the start: 2 copper layers, 55 x 40 mm, 43 parts, among them J1 Conn_01x07_Socket, Q1 2N7002, Q2 2N7002, Q3 2N7002, SW1 SW_Push, U1 NRF24L01, U2 AMS1117-3.3, U3 STM32L412KBTx, Y1 16 MHz

Commit message: Updated Schematic & PCB (Text / Miscellaneous / Antenna WIP)
Other:
- board text added: "B"
- board text added: "T"
Changed lines of the file:
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@@
     (fp_line (start 1 0.45) (end -1 0.45)
       (stroke (width 0.1) (type solid)) (layer "F.Fab"))
-    (pad "1" smd roundrect (at -1.15 0 180) (size 1.05 1.2) (layers "F.Cu" "F.Paste" "F.Mask") (roundrect_rratio 0.238095)
+    (pad "1" smd roundrect (at -1.15 0 180) (size 1.05 1.2) (layers "F.Cu" "F.Paste" "F.Mask") (roundrect_rratio 0.2380952381)
       (net 19 "ANT1") (pintype "passive"))
-    (pad "2" smd roundrect (at 1.15 0 180) (size 1.05 1.2) (layers "F.Cu" "F.Paste" "F.Mask") (roundrect_rratio 0.238095)
+    (pad "2" smd roundrect (at 1.15 0 180) (size 1.05 1.2) (layers "F.Cu" "F.Paste" "F.Mask") (roundrect_rratio 0.2380952381)
       (net 5 "VDD_PA") (pintype "passive"))
     (model "${KICAD6_3DMODEL_DIR}/Inductor_SMD.3dshapes/L_0805_2012Metric.wrl"
@@
     (fp_line (start 2 2) (end -2 2)
       (stroke (width 0.1) (type solid)) (layer "F.Fab"))
-    (pad "" smd roundrect (at -0.625 -0.625) (size 1.01 1.01) (layers "F.Paste") (roundrect_rratio 0.247525))
-    (pad "" smd roundrect (at -0.625 0.625) (size 1.01 1.01) (layers "F.Paste") (roundrect_rratio 0.247525))
-    (pad "" smd roundrect (at 0.625 -0.625) (size 1.01 1.01) (layers "F.Paste") (roundrect_rratio 0.247525))
-    (pad "" smd roundrect (at 0.625 0.625) (size 1.01 1.01) (layers "F.Paste") (roundrect_rratio 0.247525))
+    (pad "" smd roundrect (at -0.625 -0.625) (size 1.01 1.01) (layers "F.Paste") (roundrect_rratio 0.2475247525))
+    (pad "" smd roundrect (at -0.625 0.625) (size 1.01 1.01) (layers "F.Paste") (roundrect_rratio 0.2475247525))
+    (pad "" smd roundrect (at 0.625 -0.625) (size 1.01 1.01) (layers "F.Paste") (roundrect_rratio 0.2475247525))
+    (pad "" smd roundrect (at 0.625 0.625) (size 1.01 1.01) (layers "F.Paste") (roundrect_rratio 0.2475247525))
     (pad "1" smd roundrect (at -1.9375 -1) (size 0.825 0.25) (layers "F.Cu" "F.Paste" "F.Mask") (roundrect_rratio 0.25)
       (net 25 "Chip_Enable") (pinfunction "CE") (pintype "input"))
@@
     (fp_line (start 1 0.45) (end -1 0.45)
       (stroke (width 0.1) (type solid)) (layer "F.Fab"))
-    (pad "1" smd roundrect (at -1.15 0) (size 1.05 1.2) (layers "F.Cu" "F.Paste" "F.Mask") (roundrect_rratio 0.238095)
+    (pad "1" smd roundrect (at -1.15 0) (size 1.05 1.2) (layers "F.Cu" "F.Paste" "F.Mask") (roundrect_rratio 0.2380952381)
       (net 18 "ANT2") (pintype "passive"))
-    (pad "2" smd roundrect (at 1.15 0) (size 1.05 1.2) (layers "F.Cu" "F.Paste" "F.Mask") (roundrect_rratio 0.238095)
+    (pad "2" smd roundrect (at 1.15 0) (size 1.05 1.2) (layers "F.Cu" "F.Paste" "F.Mask") (roundrect_rratio 0.2380952381)
       (net 6 "Net-(C8-Pad2)") (pintype "passive"))
     (model "${KICAD6_3DMODEL_DIR}/Inductor_SMD.3dshapes/L_0805_2012Metric.wrl"
@@
     (fp_line (start 1 0.45) (end -1 0.45)
       (stroke (width 0.1) (type solid)) (layer "F.Fab"))
-    (pad "1" smd roundrect (at -1.15 0) (size 1.05 1.2) (layers "F.Cu" "F.Paste" "F.Mask") (roundrect_rratio 0.238095)
+    (pad "1" smd roundrect (at -1.15 0) (size 1.05 1.2) (layers "F.Cu" "F.Paste" "F.Mask") (roundrect_rratio 0.2380952381)
       (net 18 "ANT2") (pintype "passive"))
-    (pad "2" smd roundrect (at 1.15 0) (size 1.05 1.2) (layers "F.Cu" "F.Paste" "F.Mask") (roundrect_rratio 0.238095)
+    (pad "2" smd roundrect (at 1.15 0) (size 1.05 1.2) (layers "F.Cu" "F.Paste" "F.Mask") (roundrect_rratio 0.2380952381)
       (net 19 "ANT1") (pintype "passive"))
     (model "${KICAD6_3DMODEL_DIR}/Inductor_SMD.3dshapes/L_0805_2012Metric.wrl"
@@
   (gr_line (start 48 58) (end 93 58)
     (stroke (width 0.05) (type default)) (layer "Edge.Cuts"))
+  (gr_text "T" (at 53 61) (layer "F.Cu")
+    (effects (font (size 1.5 1.5) (thickness 0.3) bold) (justify left bottom))
+  )
+  (gr_text "B" (at 53 61) (layer "B.Cu")
+    (effects (font (size 1.5 1.5) (thickness 0.3) bold) (justify left bottom))
+  )
   (segment (start 87.1375 72.5) (end 87.1375 70.5) (width 0.3) (layer "F.Cu") (net 1))
   (segment (start 53.5875 74) (end 49.5 74) (width 0.3) (layer "F.Cu") (net 2))
