File: Hardware/Kicad/Kicad_Receptor/nRF24 extern/RecepteurSNES-ModuleNRF24ext.kicad_pcb (KiCad board)
At the start: 2 copper layers, 27 parts, among them J1 Conn_01x07_Socket, J2 Conn_01x08_Socket, Q1 2N7002, Q2 2N7002, Q3 2N7002, SW1 SW_Push, U1 STM32L412KBTx, U2 AMS1117-3.3

Commit message: Correction of the last commit
Parts:
- removed D2: LED_Small, Diode_SMD:D_0603_1608Metric_Pad1.05x0.95mm_HandSolder
- removed R2: 1k, Resistor_SMD:R_0603_1608Metric_Pad0.98x0.95mm_HandSolder
- added C3: 1u, Capacitor_SMD:C_0603_1608Metric_Pad1.08x0.95mm_HandSolder, F.Cu at (156.6, 92.0)
- added C4: 10n, Capacitor_SMD:C_0603_1608Metric_Pad1.08x0.95mm_HandSolder, F.Cu at (156.6, 93.5)
- added L1: 39n, Inductor_SMD:L_0805_2012Metric_Pad1.05x1.20mm_HandSolder, F.Cu at (156.5, 90.5)
Connections:
- U1 pad 23: Player2_LED -> unconnected-(U1-PA13-Pad23)
Routing:
- net +3.3V: track 78.6 -> 89.9 mm
- net +3.3VA: track 0.00 -> 8.86 mm, vias 0 -> 2
- net Player2_LED: track 2.14 -> 0.00 mm
- net Net-(D2-K): track 1.62 -> 0.00 mm
- net GND: track 84.8 -> 86.3 mm
- added copper zone on B.Cu, net GND
- added copper zone on F.Cu, net GND
