File: Hardware/Kicad/Kicad_Receptor/nRF24 extern/RecepteurSNES-ModuleNRF24ext.kicad_sch (KiCad schematic)
At the start: 27 parts, among them J1 Conn_01x07_Socket, J2 Conn_01x08_Socket, Q1 2N7002, Q2 2N7002, Q3 2N7002, SW1 SW_Push, U2 AMS1117-3.3, U3 STM32L412KBTx

Commit message: Correction of the last commit
Parts:
- removed D1: LED_Small, Diode_SMD:D_0603_1608Metric_Pad1.05x0.95mm_HandSolder, symbol Device:LED_Small
- removed R9: 1k, Resistor_SMD:R_0603_1608Metric_Pad0.98x0.95mm_HandSolder, symbol Device:R_Small
- added C5: 1u, Capacitor_SMD:C_0603_1608Metric_Pad1.08x0.95mm_HandSolder, symbol Device:C_Small
- added C6: 10n, Capacitor_SMD:C_0603_1608Metric_Pad1.08x0.95mm_HandSolder, symbol Device:C_Small
- added L1: 39n, Inductor_SMD:L_0805_2012Metric_Pad1.05x1.20mm_HandSolder, symbol Device:L_Small
Connections:
- net +3.3V: now also L1.1
- net +3.3VA: now also C5.1, C6.1, L1.2
- net GND: now also C5.2, C6.2
- net Player2_LED: no longer names the net of U3.23 (PA13)
- no-connect marks 18 -> 19
Other:
- moved on the sheet: C1, C2, J1, J2, Q1, Q2, Q3, R3, R4, R5, R6, R7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
