File: Hardware/Kicad/NRF24L01_Include/SNES_Controller_NRF24L01_Include.kicad_sch (KiCad schematic)
At the start: 43 parts, among them J1 Conn_01x07_Socket, Q1 2N7002, Q2 2N7002, Q3 2N7002, SW1 SW_Push, U1 NRF24L01, U2 AMS1117-3.3, U3 STM32L412KBTx, Y1 16 MHz

Commit message: Updated NRF24L01 (Exclude & Include) Kicad projects to revision 2.0
Other:
- title: Wireless SNES Receiver -> SNES Wireless Receiver (NRF24L01 Include)
