File: Hardware/Kicad/Controller/Projet_manette_proto.kicad_sch (KiCad schematic)
At the start: 67 parts, among them J1 Conn_01x02, SW1 SW_Push, SW10 SW_Push, SW11 SW_DIP_x01, SW12 SW_Push, SW13 SW_DIP_x01, SW2 SW_Push, SW3 SW_Push, SW4 SW_Push, SW5 SW_Push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

Commit message: CONTROLER V1
Connections:
- net GND: no longer U1.10 (PA4), U1.11 (PA5), U1.12 (PA6), U1.13 (PA7), U1.18 (PA8), U1.19 (PA9), U1.23 (PA13), U1.6 (PA0), U1.7 (PA1), U1.8 (PA2), U1.9 (PA3)
- net UC_Button: now reaches R5.1, SW5.1
- net UC_Button: now also U1.10 (PA4)
- net X_Button: now reaches R3.1, SW3.1
- net X_Button: now also U1.8 (PA2)
- net SE_Button: now reaches R10.1, SW10.1
- net SE_Button: now also U1.19 (PA9)
- net Y_Button: now reaches R4.1, SW4.1
- net Y_Button: now also U1.9 (PA3)
- net DC_Button: now reaches R8.1, SW8.1
- net DC_Button: now also U1.11 (PA5)
- net A_Button: now reaches R1.1, SW1.1
- net A_Button: now also U1.6 (PA0)
- net ST_Button: now reaches R9.1, SW9.1
- net ST_Button: now also U1.18 (PA8)
- net LC_Button: now reaches R6.1, SW6.1
- net LC_Button: now also U1.12 (PA6)
- net B_Button: now reaches R2.1, SW2.1
- net B_Button: now also U1.7 (PA1)
- net NES/SNES_switcher: now reaches R19.1, SW13.1
- net NES/SNES_switcher: now also U1.23 (PA13)
- net RC_Button: now reaches R7.1, SW7.1
- net RC_Button: now also U1.13 (PA7)
Other:
- moved on the sheet: R1, R10, R19, R2, R3, R4, R5, R6, R7, R8, R9
