File: Hardware/Kicad/NRF24L01_Exclude/NRF24L01_Exclude.kicad_pcb (KiCad board)
At the start: 2 copper layers, 30 x 32.5 mm, 28 parts, among them J1 Conn_01x07_Socket, J2 Conn_01x08_Socket, Q1 2N7002, Q2 2N7002, Q3 2N7002, SW1 SW_Push, U1 STM32L412KBTx, U2 AMS1117-3.3

Commit message: correction
Routing:
- net +3.3V: track 68.1 -> 70.7 mm
Changed lines of the file:
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@@
   (segment (start 138.65 103.325) (end 139.175 102.8) (width 0.3) (layer "F.Cu") (net 3))
   (segment (start 127.7 104.175) (end 127.25 103.725) (width 0.3) (layer "F.Cu") (net 3))
+  (segment (start 140.4505 103.2) (end 139.575 103.2) (width 0.3) (layer "F.Cu") (net 3))
+  (segment (start 129.52 110.28) (end 127.7 108.46) (width 0.3) (layer "F.Cu") (net 3))
+  (segment (start 144.15 98) (end 144.5 97.65) (width 0.3) (layer "F.Cu") (net 3))
+  (segment (start 127.7 108.46) (end 127.7 104.175) (width 0.3) (layer "F.Cu") (net 3))
   (segment (start 144.5 97.65) (end 144.5 91.35) (width 0.3) (layer "F.Cu") (net 3))
-  (segment (start 129.52 110.28) (end 127.7 108.46) (width 0.3) (layer "F.Cu") (net 3))
-  (segment (start 127.7 108.46) (end 127.7 104.175) (width 0.3) (layer "F.Cu") (net 3))
   (segment (start 134.0875 90.5475) (end 134.05 90.51) (width 0.3) (layer "F.Cu") (net 3))
   (segment (start 127.25 94.3625) (end 127.8625 93.75) (width 0.3) (layer "F.Cu") (net 3))
@@
   (segment (start 130.745 110.28) (end 129.52 110.28) (width 0.3) (layer "F.Cu") (net 3))
   (segment (start 137.5875 93.75) (end 137.5875 90.5475) (width 0.3) (layer "F.Cu") (net 3))
+  (segment (start 141.8 98) (end 144.15 98) (width 0.3) (layer "F.Cu") (net 3))
   (segment (start 130.5875 93.75) (end 130.5875 90.5475) (width 0.3) (layer "F.Cu") (net 3))
   (segment (start 137.5875 90.5475) (end 137.55 90.51) (width 0.3) (layer "F.Cu") (net 3))
   (segment (start 127.8625 93.75) (end 130.5875 93.75) (width 0.3) (layer "F.Cu") (net 3))
+  (segment (start 139.575 103.2) (end 139.175 102.8) (width 0.3) (layer "F.Cu") (net 3))
   (via (at 134.05 90.51) (size 0.8) (drill 0.4) (layers "F.Cu" "B.Cu") (net 3))
-  (via (at 139.175 102.8995) (size 0.8) (drill 0.4) (layers "F.Cu" "B.Cu") (net 3))
-  (via (at 144.5 97.65) (size 0.8) (drill 0.4) (layers "F.Cu" "B.Cu") (net 3))
+  (via (at 140.4505 103.2) (size 0.8) (drill 0.4) (layers "F.Cu" "B.Cu") (net 3))
+  (via (at 141.8 98) (size 0.8) (drill 0.4) (layers "F.Cu" "B.Cu") (net 3))
   (via (at 144.5 91.35) (size 0.8) (drill 0.4) (layers "F.Cu" "B.Cu") (net 3))
   (via (at 130.55 90.51) (size 0.8) (drill 0.4) (layers "F.Cu" "B.Cu") (net 3))
   (via (at 137.55 90.51) (size 0.8) (drill 0.4) (layers "F.Cu" "B.Cu") (net 3))
   (segment (start 134.05 90.51) (end 130.55 90.51) (width 0.3) (layer "B.Cu") (net 3))
+  (segment (start 140.4505 101.6995) (end 141.8 100.35) (width 0.3) (layer "B.Cu") (net 3))
   (segment (start 143.66 90.51) (end 144.5 91.35) (width 0.3) (layer "B.Cu") (net 3))
-  (segment (start 144.5 97.65) (end 139.2505 102.8995) (width 0.3) (layer "B.Cu") (net 3))
-  (segment (start 139.2505 102.8995) (end 139.175 102.8995) (width 0.3) (layer "B.Cu") (net 3))
+  (segment (start 141.8 100.35) (end 141.8 98) (width 0.3) (layer "B.Cu") (net 3))
+  (segment (start 140.4505 103.2) (end 140.4505 101.6995) (width 0.3) (layer "B.Cu") (net 3))
   (segment (start 137.55 90.51) (end 143.66 90.51) (width 0.3) (layer "B.Cu") (net 3))
   (segment (start 137.55 90.51) (end 134.05 90.51) (width 0.3) (layer "B.Cu") (net 3))
