File: Hardware/Kicad/NRF24L01_Exclude/NRF24L01_Exclude.kicad_sch (KiCad schematic)
At the start: 28 parts, among them J1 Conn_01x07_Socket, J2 Conn_01x08_Socket, Q1 2N7002, Q2 2N7002, Q3 2N7002, SW1 SW_Push, U2 AMS1117-3.3, U3 STM32L412KBTx

Commit message: correction
Parts:
- removed C5: 1u, Capacitor_SMD:C_0603_1608Metric_Pad1.08x0.95mm_HandSolder, symbol Device:C_Small
- removed C6: 10n, Capacitor_SMD:C_0603_1608Metric_Pad1.08x0.95mm_HandSolder, symbol Device:C_Small
- removed L1: 39n, Inductor_SMD:L_0805_2012Metric_Pad1.05x1.20mm_HandSolder, symbol Device:L_Small
Connections:
- net +3.3VA is gone; now on net +3.3V: U3.5 (VDDA)
