File: Hardware/Kicad/Plug_NRF24L01_Include (Backup)/Plug_NRF24L01_Include.kicad_sch (KiCad schematic)
At the start: 54 parts, among them J1 Conn_01x07_Socket, J2 Conn_02x07_Odd_Even, Q1 2N7002, Q2 2N7002, Q3 2N7002, Q4 2N7002, Q5 2N7002, SW2 SW_SPST, U1 STM32L412KBTx, U2 MIC5219-3.3YMM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

Commit message: Updated Plug_NRF24L01_Include. Schematic (Pins assignment / Appairing Button). PCB (Finalized routing / Antenna not working).
Connections:
- net Appairing_Btn: now also U1.2 (PC14); no longer U1.10 (PA4)
- net Chip_Enable: now also U1.11 (PA5); no longer U1.15 (PB1)
- net Data_Clock_SNES: now also Q2.3 (D), R13.2; no longer Q1.3 (D), R12.2
- net Data_Clock_STM32: now also Q2.2 (S), R8.2, U1.29 (PB6); no longer Q1.2 (S), R7.2, U1.26 (PB3)
- net Data_Latch_SNES: now also Q3.3 (D), R14.2; no longer Q2.3 (D), R13.2
- net Data_Latch_STM32: now also Q3.2 (S), R9.2; no longer Q2.2 (S), R8.2
- net GND: no longer C9.2, J1.7 (Pin_7), R1.2, U3.14 (VSS), U3.17 (VSS), U3.20 (VSS), U3.8 (VSS)
- net IOBit_SNES: now also Q4.3 (D), R15.2; no longer Q5.3 (D), R16.2
- net IOBit_STM32: now also Q4.2 (S), R10.2; no longer Q5.2 (S), R11.2
- net NRST: now also J2.12 (Pin_12); no longer J2.6 (Pin_6)
- net Player1_LED: now also U1.20 (PA10); no longer U1.23 (PA13)
- net SPI_Chip_Select: now also U1.7 (PA1); no longer U1.14 (PB0)
- net SPI_Clock: now also U1.6 (PA0); no longer U1.13 (PA7)
- net SPI_Digital_Output: now also U1.10 (PA4); no longer U1.11 (PA5)
- net SWDCK: now also J2.6 (Pin_6), U1.24 (PA14); no longer J2.10 (Pin_10), U1.7 (PA1)
- net SWDIO: now also J2.4 (Pin_4), U1.23 (PA13); no longer J2.8 (Pin_8), U1.6 (PA0)
- net Serial_Data1_SNES: now also Q1.3 (D), R12.2; no longer Q3.3 (D), R14.2
- net Serial_Data1_STM32: now also Q1.2 (S), R7.2, U1.25 (PA15); no longer Q3.2 (S), R9.2, U1.28 (PB5)
- net Serial_Data2_SNES: now also Q5.3 (D), R16.2; no longer Q4.3 (D), R15.2
- net Serial_Data2_STM32: now also Q5.2 (S), R11.2, U1.28 (PB5); no longer Q4.2 (S), R10.2, U1.29 (PB6)
- net Status_LED: now also U1.19 (PA9); no longer U1.24 (PA14)
- net USART2_RX: now also J2.13 (Pin_13), U1.9 (PA3); no longer J2.12 (Pin_12), U1.8 (PA2)
- net USART2_TX: now also U1.8 (PA2); no longer U1.9 (PA3)
- new net GND1: C9.2, R1.2, U3.14 (VSS), U3.17 (VSS), U3.20 (VSS), U3.8 (VSS)
- new net GND3: J1.7 (Pin_7)
