File: Hardware/Kicad/Controller_NRF24L01_Include/Controller_NRF24L01_Include.kicad_pcb (KiCad board)
At the start: 2 copper layers, 180 x 75 mm, 67 parts, among them J1 Conn_01x02, SW1 SW_Push, SW10 SW_Push, SW11 SW_DIP_x01, SW12 SW_Push, SW13 SW_DIP_x01, SW2 SW_Push, SW3 SW_Push, SW4 SW_Push, SW5 SW_Push, SW6 SW_Push, SW7 SW_Push, SW8 SW_Push, SW9 SW_Push, U1 STM32L412KBTx, U2 MIC5219-3.3YMM, U3 NRF24L01, Y1 16MHz

Commit message: L ET RRRRRRRRRRRRRRRRRRRRRR
Parts:
- Y1: footprint Oscillator:Oscillator_SMD_EuroQuartz_XO91-4Pin_7.0x5.0mm -> Crystal:Crystal_SMD_HC49-SD_HandSoldering
- moved Y1 4.19 mm to (138.5, 61.0)
Routing:
- net Glob_Alim: track 341.4 -> 355.9 mm
- net Net-(U3-XC1): track 44.1 -> 51.5 mm
- net Net-(U3-XC2): track 36.1 -> 38.5 mm

Commit message: correction
Parts:
- J1, U3: moved to F.Cu
- moved H6 103.3 mm to (173.7, 74.6)
- moved H5 100.2 mm to (173.7, 67.5)
- moved SW1 91.0 mm to (126.2, 65.9)
- moved R1 89.0 mm to (135.1, 104.4)
- moved R3 85.4 mm to (135.1, 109.4)
- moved C13 85.0 mm to (130.7, 111.9), turned to 0 degrees
- moved H1 84.4 mm to (159.4, 67.5)
- moved SW3 82.5 mm to (126.2, 83.0)
- moved C12 81.7 mm to (130.7, 109.4), turned to 0 degrees
- moved SW2 81.5 mm to (126.2, 74.5)
- moved R2 78.0 mm to (135.1, 106.9)
- moved R4 74.8 mm to (135.1, 111.9)
- moved SW4 73.4 mm to (126.2, 91.6)
- moved H3 70.6 mm to (166.6, 67.5)
- moved D6 68.5 mm to (148.2, 112.3), turned to 0 degrees
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Routing:
- net Glob_Alim: track 355.9 -> 0.00 mm, vias 11 -> 0
- net GND: track 185.2 -> 0.00 mm, vias 7 -> 0
- net A_Button: track 109.6 -> 0.00 mm
- net LC_Button: track 107.8 -> 0.00 mm, vias 2 -> 0
- net X_Button: track 93.3 -> 0.00 mm
- net B_Button: track 89.0 -> 0.00 mm
- net UC_Button: track 85.2 -> 0.00 mm, vias 2 -> 0
- net Y_Button: track 79.6 -> 0.00 mm, vias 2 -> 0
- net DC_Button: track 78.3 -> 0.00 mm, vias 2 -> 0
- net RC_Button: track 74.2 -> 0.00 mm, vias 2 -> 0
- net Li-ion: track 54.0 -> 0.00 mm
- net Net-(U3-XC1): track 51.5 -> 0.00 mm, vias 3 -> 0
- net NES/SNES_switcher: track 45.8 -> 0.00 mm, vias 2 -> 0
- net Net-(U3-XC2): track 38.5 -> 0.00 mm, vias 3 -> 0
- net Order_Search: track 37.8 -> 0.00 mm, vias 2 -> 0
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Other:
- board outline removed

Commit message: Thanks M.Papazoglou,more led, more Software problem
Parts:
- removed SW12: SW_Push, Button_Switch_THT:SW_PUSH_6mm_H5mm
- added J2: Conn_02x07_Odd_Even, Connector_PinHeader_1.27mm:PinHeader_2x07_P1.27mm_Vertical_SMD, F.Cu at (125.5, 22.4)
- added R20: 1K, Resistor_SMD:R_0603_1608Metric_Pad0.98x0.95mm_HandSolder, F.Cu at (127.5, 33.1)
- added R21: 1K, Resistor_SMD:R_0603_1608Metric_Pad0.98x0.95mm_HandSolder, F.Cu at (127.5, 35.6)
- added SW14: SW_SPST, Button_Switch_SMD:SW_SPST_B3S-1000, F.Cu at (55.0, 45.5)
- added TP1: R, Connector_Coaxial:SMA_Molex_73251-1153_EdgeMount_Horizontal, F.Cu at (95.5, 65.8)
- added TP2: L, Connector_Coaxial:SMA_Molex_73251-1153_EdgeMount_Horizontal, F.Cu at (184.5, 65.3)
- C2: value 4.7nF -> 4.7pF; footprint Capacitor_SMD:C_0603_1608Metric_Pad1.08x0.95mm_HandSolder -> Capacitor_SMD:C_0402_1005Metric_Pad0.74x0.62mm_HandSolder
- C3: footprint Capacitor_SMD:C_0603_1608Metric_Pad1.08x0.95mm_HandSolder -> Capacitor_SMD:C_0402_1005Metric_Pad0.74x0.62mm_HandSolder
- C4: value 1.5nF -> 1.5pF; footprint Capacitor_SMD:C_0603_1608Metric_Pad1.08x0.95mm_HandSolder -> Capacitor_SMD:C_0402_1005Metric_Pad0.74x0.62mm_HandSolder
- C5: value 1.0nF -> 1.0pF; footprint Capacitor_SMD:C_0603_1608Metric_Pad1.08x0.95mm_HandSolder -> Capacitor_SMD:C_0402_1005Metric_Pad0.74x0.62mm_HandSolder
- L2: value 2.7nF -> 2.7nH; footprint Inductor_SMD:L_0603_1608Metric_Pad1.05x0.95mm_HandSolder -> Inductor_SMD:L_0402_1005Metric_Pad0.77x0.64mm_HandSolder
- L3: value 8.2nF -> 8.2nH
- SW1, SW10, SW2, SW3, SW4, SW5, SW6, SW7, SW8, SW9: value SW_Push -> SW_SPST; footprint Button_Switch_THT:SW_PUSH_6mm_H5mm -> Button_Switch_SMD:SW_SPST_B3S-1000
- moved SW1 130.2 mm to (254.4, 89.1)
- moved SW3 127.3 mm to (253.5, 78.8)
- moved SW2 115.3 mm to (240.6, 88.8)
- moved SW4 114.8 mm to (240.2, 78.3)
- moved SW6 102.0 mm to (35.0, 80.6)
- moved SW7 102.0 mm to (35.0, 89.0)
- moved SW8 102.0 mm to (35.0, 97.5)
- moved SW10 99.6 mm to (55.0, 37.1)
- moved SW9 99.6 mm to (55.0, 28.6)
- moved H2 97.7 mm to (68.0, 109.0)
- moved H1 91.4 mm to (68.0, 67.0)
- moved C1 75.2 mm to (151.1, 28.4)
- moved C10 75.2 mm to (155.4, 33.4)
- moved C11 75.2 mm to (155.4, 35.9)
- moved C12 75.2 mm to (155.4, 38.4)
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Connections:
- SW1 pad 1: A_Button -> B_Button
- SW10 pad 1: SE_Button -> Order_Search
- SW2 pad 1: B_Button -> X_Button
- SW3 pad 1: X_Button -> Y_Button
- SW4 pad 1: Y_Button -> UC_Button
- SW5 pad 1: UC_Button -> LC_Button
- SW6 pad 1: LC_Button -> RC_Button
- SW7 pad 1: RC_Button -> DC_Button
- SW8 pad 1: DC_Button -> ST_Button
- SW9 pad 1: ST_Button -> SE_Button
- U1 pad 15: unconnected-(U1-PB1-Pad15) -> NES/SNES_switcher
- U1 pad 2: unconnected-(U1-PC14-Pad2) -> Y_Button
- U1 pad 23: NES/SNES_switcher -> SWDIO
- U1 pad 24: unconnected-(U1-PA14-Pad24) -> SWDCK
- U1 pad 29: unconnected-(U1-PB6-Pad29) -> R
- U1 pad 3: unconnected-(U1-PC15-Pad3) -> X_Button
- U1 pad 30: unconnected-(U1-PB7-Pad30) -> L
- U1 pad 4: unconnected-(U1-NRST-Pad4) -> Reset_Buton 
- U1 pad 8: X_Button -> USART2_TX
- U1 pad 9: Y_Button -> USART2_RX
Routing:
- removed copper zone on B.Cu, net GND

Commit message: New controler versions, and not the last
Parts:
- removed the C12 at (155.4, 38.4)
- removed the D2 at (172.9, 31.0)
- removed the R1 at (159.8, 33.4)
- removed the R2 at (159.8, 35.9)
- removed the R3 at (159.8, 38.4)
- removed the R4 at (159.8, 40.9)
- removed the R5 at (159.8, 43.4)
- removed the SW1 at (254.4, 89.1)
- removed SW14: SW_SPST, Button_Switch_SMD:SW_SPST_B3S-1000
- removed the SW7 at (35.0, 89.0)
- added C13: 1nF, Capacitor_SMD:C_0603_1608Metric_Pad1.08x0.95mm_HandSolder, F.Cu at (105.3, -58.8)
- added D10: G7, LED_SMD:LED_0603_1608Metric_Pad1.05x0.95mm_HandSolder, F.Cu at (45.8, -30.6)
- added D11: G8, LED_SMD:LED_0603_1608Metric_Pad1.05x0.95mm_HandSolder, F.Cu at (57.7, -30.6)
- added D12: O1, LED_SMD:LED_0603_1608Metric_Pad1.05x0.95mm_HandSolder, F.Cu at (69.7, -30.6)
- added D13: O2, LED_SMD:LED_0603_1608Metric_Pad1.05x0.95mm_HandSolder, F.Cu at (81.6, -30.6)
- added D14: O3, LED_SMD:LED_0603_1608Metric_Pad1.05x0.95mm_HandSolder, F.Cu at (93.5, -30.6)
- added D15: O4, LED_SMD:LED_0603_1608Metric_Pad1.05x0.95mm_HandSolder, F.Cu at (33.9, -3.44)
- added D16: R1, LED_SMD:LED_0603_1608Metric_Pad1.05x0.95mm_HandSolder, F.Cu at (45.8, -3.44)
- added D17: R2, LED_SMD:LED_0603_1608Metric_Pad1.05x0.95mm_HandSolder, F.Cu at (57.7, -3.44)
- added D18: R3, LED_SMD:LED_0603_1608Metric_Pad1.05x0.95mm_HandSolder, F.Cu at (69.7, -3.44)
- added D19: R4, LED_SMD:LED_0603_1608Metric_Pad1.05x0.95mm_HandSolder, F.Cu at (81.6, -3.44)
- added D7: G4, LED_SMD:LED_0603_1608Metric_Pad1.05x0.95mm_HandSolder, F.Cu at (81.6, -57.8)
- added D8: G5, LED_SMD:LED_0603_1608Metric_Pad1.05x0.95mm_HandSolder, F.Cu at (93.5, -57.8)
- added D9: G6, LED_SMD:LED_0603_1608Metric_Pad1.05x0.95mm_HandSolder, F.Cu at (33.9, -30.6)
- added R11: 1K, Resistor_SMD:R_0603_1608Metric_Pad0.98x0.95mm_HandSolder, F.Cu at (105.3, -43.7)
- added R12: 1K, Resistor_SMD:R_0603_1608Metric_Pad0.98x0.95mm_HandSolder, F.Cu at (105.3, -41.2)
- added R19: 1K, Resistor_SMD:R_0603_1608Metric_Pad0.98x0.95mm_HandSolder, F.Cu at (109.7, -43.7)
- added R20: 1K, Resistor_SMD:R_0603_1608Metric_Pad0.98x0.95mm_HandSolder, F.Cu at (109.7, -41.2)
- added R21: 1K, Resistor_SMD:R_0603_1608Metric_Pad0.98x0.95mm_HandSolder, F.Cu at (114.0, -58.8)
- added R22: 1K, Resistor_SMD:R_0603_1608Metric_Pad0.98x0.95mm_HandSolder, F.Cu at (114.0, -56.3)
- added R23: 1K, Resistor_SMD:R_0603_1608Metric_Pad0.98x0.95mm_HandSolder, F.Cu at (114.0, -53.8)
- added R24: 1K, Resistor_SMD:R_0603_1608Metric_Pad0.98x0.95mm_HandSolder, F.Cu at (114.0, -51.2)
- added R25: 1K, Resistor_SMD:R_0603_1608Metric_Pad0.98x0.95mm_HandSolder, F.Cu at (114.0, -48.7)
- added R26: 1K, Resistor_SMD:R_0603_1608Metric_Pad0.98x0.95mm_HandSolder, F.Cu at (114.0, -46.2)
- added SW11: SW_SPST, Button_Switch_SMD:SW_SPST_B3S-1000, F.Cu at (134.8, -38.9)
- added SW12: SW_SPST, Button_Switch_SMD:SW_SPST_B3S-1000, F.Cu at (134.8, -30.4)
- added SW13: SW_SPST, Button_Switch_SMD:SW_SPST_B3S-1000, F.Cu at (134.8, -22.0)
- added U4: PCA9685PW, Package_SO:TSSOP-28_4.4x9.7mm_P0.65mm, F.Cu at (107.5, -34.3)
- D3: value LED -> D_Small; footprint LED_SMD:LED_0603_1608Metric_Pad1.05x0.95mm_HandSolder -> Display:HDSP-4832
- D4: value LED -> G1
- D5: value LED -> G2
- D6: value LED -> G3
- R10, R8, R9: value 1K -> 10K
- R14, R15, R16, R17: value R_Small -> 1K
- R6, R7: value 1K -> 1M
- moved SW2 185.9 mm to (123.8, -55.8)
- moved SW3 181.0 mm to (123.8, -47.4)
- moved D3 166.3 mm to (33.9, -57.8)
- moved SW4 165.2 mm to (123.8, -38.9)
- moved D4 158.0 mm to (45.8, -57.8)
- moved D5 150.3 mm to (57.7, -57.8)
- moved D6 143.1 mm to (69.7, -57.8)
- moved SW6 135.7 mm to (123.8, -22.0)
- moved SW5 111.1 mm to (123.8, -30.4)
- moved SW9 110.2 mm to (134.8, -47.4)
- moved R13 105.1 mm to (109.7, -58.8)
- moved R14 105.1 mm to (109.7, -56.3)
- moved R15 105.1 mm to (109.7, -53.8)
- moved R16 105.1 mm to (109.7, -51.2)
- moved R17 105.1 mm to (109.7, -48.7)
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- renumbered C10 to C1, C1 to C10, C3 to C11, C2 to C12, C8 to C2, C9 to C3, C13 to C4, C4 to C5, C5 to C6, C6 to C7, C7 to C8, C11 to C9, D7 to D1, D1 to D2, L3 to L1, L1 to L2, L2 to L3, R12 to R1, R11 to R2, R19 to R3, R20 to R4, R21 to R5, SW11 to SW1, SW13 to SW10, SW10 to SW7, U3 to U2, U2 to U3
Connections:
- D3 pad 1: GND -> Net-(D3-K)
- D3 pad 2: Net-(D3-A) -> Glob_Alim
- D4 pad 1: GND -> Net-(D4-K)
- D5 pad 1: GND -> Net-(D5-K)
- D6 pad 1: GND -> Net-(D6-K)
- R10 pad 1: SE_Button -> DIODE_OE
- R10 pad 2: GND -> Glob_Alim
- R13 pad 1: Order_Search -> Net-(D6-K)
- R14 pad 1: Li-ion -> Net-(D7-K)
- R14 pad 2: Net-(D5-A) -> GND
- R15 pad 1: Li-ion -> Net-(D8-K)
- R15 pad 2: Net-(D3-A) -> GND
- R16 pad 1: Li-ion -> Net-(D9-K)
- R16 pad 2: Net-(D4-A) -> GND
- R17 pad 1: Li-ion -> Net-(D10-K)
- R17 pad 2: Net-(D6-A) -> GND
- R6 pad 1: LC_Button -> Li-ion
- R6 pad 2: GND -> POWER_CHECK
- R7 pad 1: RC_Button -> POWER_CHECK
- R8 pad 1: DC_Button -> DIODE_SDA
- R8 pad 2: GND -> Glob_Alim
- R9 pad 1: ST_Button -> Glob_Alim
- R9 pad 2: GND -> DIODE_CLK
- SW2 pad 1: X_Button -> GND
- SW2 pad 2: Glob_Alim -> A_Button
- SW3 pad 1: Y_Button -> GND
- SW3 pad 2: Glob_Alim -> B_Button
- SW4 pad 1: UC_Button -> GND
- SW4 pad 2: Glob_Alim -> X_Button
- SW5 pad 1: LC_Button -> GND
- SW5 pad 2: Glob_Alim -> Y_Button
- SW6 pad 1: RC_Button -> GND
- SW6 pad 2: Glob_Alim -> UC_Button
- SW7 pad 1: Order_Search -> GND
- SW7 pad 2: Glob_Alim -> Order_Search
- SW8 pad 1: ST_Button -> GND
- SW8 pad 2: Glob_Alim -> LC_Button
- SW9 pad 1: SE_Button -> GND
- SW9 pad 2: Glob_Alim -> RC_Button
- U1 pad 10: UC_Button -> Order_Search
- U1 pad 11: DC_Button -> Pin_Clock
- U1 pad 12: LC_Button -> Digital_Out_Put
- U1 pad 13: RC_Button -> MOSI
- U1 pad 14: unconnected-(U1-PB0-Pad14) -> POWER_CHECK
- U1 pad 15: NES/SNES_switcher -> RC_Button
- U1 pad 20: Order_Search -> DIODE_CLK
- U1 pad 22: LED_Order -> DIODE_SDA
- U1 pad 25: unconnected-(U1-PA15-Pad25) -> DIODE_OE
- U1 pad 26: Pin_Clock -> LC_Button
- U1 pad 27: Digital_Out_Put -> DC_Button
- U1 pad 28: MOSI -> UC_Button
- U1 pad 31: unconnected-(U1-PH3-Pad31) -> NES/SNES_switcher
Routing:
- added copper zone on B.Cu, net GND

Commit message: New New controler vers
Parts:
- D3: footprint Display:HDSP-4832 -> LED_SMD:LED_0603_1608Metric_Pad1.05x0.95mm_HandSolder
- J1: moved to B.Cu
- moved C13 189.9 mm to (196.5, 107.8), turned to -90 degrees
- moved R6 184.8 mm to (196.5, 104.5), turned to -90 degrees
- moved R7 184.8 mm to (195.0, 107.8), turned to -90 degrees
- moved D3 179.5 mm to (159.7, 70.3)
- moved H6 165.7 mm to (68.1, 87.0)
- moved SW2 161.0 mm to (198.0, 87.0)
- moved SW3 158.0 mm to (188.0, 97.0)
- moved D9 151.6 mm to (150.9, 65.8), turned to -90 degrees
- moved SW9 144.4 mm to (82.0, 87.0)
- moved D15 143.8 mm to (159.9, 65.8), turned to -90 degrees
- moved D10 143.7 mm to (152.4, 65.8), turned to -90 degrees
- moved R9 137.9 mm to (160.4, 77.7), turned to 180 degrees
- moved D11 136.2 mm to (153.9, 65.8), turned to -90 degrees
- moved D8 135.6 mm to (149.4, 65.8), turned to -90 degrees
- moved D16 134.7 mm to (161.4, 65.8), turned to -90 degrees
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Routing:
- net Glob_Alim: track 0.00 -> 150.3 mm, vias 0 -> 9
- net SWDIO: track 0.00 -> 115.7 mm, vias 0 -> 2
- net SWDCK: track 0.00 -> 112.8 mm, vias 0 -> 6
- net RC_Button: track 0.00 -> 105.7 mm
- net X_Button: track 0.00 -> 83.7 mm, vias 0 -> 2
- net A_Button: track 0.00 -> 76.7 mm, vias 0 -> 2
- net Order_Search: track 0.00 -> 76.7 mm, vias 0 -> 2
- net Y_Button: track 0.00 -> 66.1 mm, vias 0 -> 4
- net B_Button: track 0.00 -> 64.6 mm, vias 0 -> 2
- net POWER_CHECK: track 0.00 -> 64.6 mm, vias 0 -> 2
- net Reset_Buton : track 0.00 -> 55.9 mm, vias 0 -> 2
- net USART2_TX: track 0.00 -> 55.8 mm, vias 0 -> 2
- net DIODE_OE: track 0.00 -> 52.7 mm, vias 0 -> 5
- net Li-ion: track 0.00 -> 51.0 mm, vias 0 -> 2
- net UC_Button: track 0.00 -> 50.8 mm
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
Commit message: New New New version of the controler include, we hope that will be the last
Parts:
- moved D19 0.70 mm to (166.6, 65.8)
- moved D18 0.58 mm to (165.0, 65.8)
- moved D17 0.48 mm to (163.4, 65.8)
- moved D8 0.48 mm to (148.9, 65.8)
- moved D16 0.38 mm to (161.8, 65.8)
- moved D9 0.38 mm to (150.5, 65.8)
- moved D10 0.28 mm to (152.1, 65.8)
- moved D15 0.28 mm to (160.2, 65.8)
- moved R2 0.20 mm to (138.8, 78.4)
- moved Y1 0.20 mm to (142.2, 78.0)
- moved D11 0.18 mm to (153.7, 65.8)
- moved D14 0.18 mm to (158.6, 65.8)
- moved D12 0.08 mm to (155.3, 65.8)
Routing:
- net GND: track 33.8 -> 64.4 mm, vias 2 -> 4

Commit message: And a new version of the controler
Parts:
- moved SW2 5.00 mm to (203.0, 87.0)
- moved SW9 5.00 mm to (77.0, 87.0)
- moved SW3 2.50 mm to (190.5, 97.0)
- moved SW4 2.50 mm to (190.5, 77.0)
- moved SW6 2.50 mm to (89.5, 77.0)
- moved SW8 2.50 mm to (89.5, 97.0)
- moved H5 0.28 mm to (213.0, 87.8)
- moved H6 0.10 mm to (68.0, 87.0)
Connections:
- Antenna_nRF1 pad 1: Antenna -> Net-(Antenna_nRF1-Feed_point)
- Antenna_nRF1 pad 2: GND -> Net-(Antenna_nRF1-GND)
Routing:
- net RC_Button: track 105.7 -> 115.4 mm
- net LC_Button: track 43.8 -> 51.7 mm
- net A_Button: track 76.7 -> 81.7 mm
- net X_Button: track 83.7 -> 86.2 mm
- net UC_Button: track 50.8 -> 53.3 mm
- net B_Button: track 64.6 -> 67.1 mm
- net Li-ion: track 51.0 -> 52.4 mm

Commit message: Maybe the final version
Parts:
- moved R5 55.9 mm to (185.1, 69.2), turned to 0 degrees
- moved SW11 17.7 mm to (89.5, 99.5)
- moved SW8 16.0 mm to (102.0, 87.0)
- moved H1 10.0 mm to (78.0, 67.0)
- moved H2 10.0 mm to (78.0, 109.0)
- moved H3 10.0 mm to (203.0, 67.0)
- moved H4 10.0 mm to (203.0, 109.0)
- moved R6 8.32 mm to (201.0, 97.5)
- moved C13 8.19 mm to (201.0, 101.0)
- moved R7 7.92 mm to (199.0, 101.0)
- moved J1 7.07 mm to (205.0, 97.0)
- moved SW3 2.69 mm to (191.5, 99.5)
- moved SW4 2.69 mm to (191.5, 74.5)
- moved SW6 2.50 mm to (89.5, 74.5)
- moved SW5 2.00 mm to (179.0, 87.0)
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Connections:
- net Reset_Buton  renamed Reset_Button 
- Antenna_nRF1 pad 1: Net-(Antenna_nRF1-Feed_point) -> Antenna
- Antenna_nRF1 pad 2: Net-(Antenna_nRF1-GND) -> GND
- U1 pad 14: POWER_CHECK -> DC_Button
- U1 pad 15: RC_Button -> UC_Button
- U1 pad 2: Y_Button -> RC_Button
- U1 pad 20: DIODE_CLK -> X_Button
- U1 pad 22: DIODE_SDA -> Y_Button
- U1 pad 26: LC_Button -> DIODE_CLK
- U1 pad 27: DC_Button -> POWER_CHECK
- U1 pad 28: UC_Button -> DIODE_SDA
- U1 pad 3: X_Button -> LC_Button
Routing:
- net L: track 23.2 -> 117.6 mm, vias 5 -> 4
- net UC_Button: track 53.3 -> 122.4 mm, vias 0 -> 4
- net DC_Button: track 36.9 -> 94.3 mm, vias 2 -> 4
- net POWER_CHECK: track 64.6 -> 109.6 mm
- net RC_Button: track 115.4 -> 84.7 mm, vias 0 -> 4
- net X_Button: track 86.2 -> 72.7 mm
- net DIODE_SDA: track 40.5 -> 51.0 mm
- net Reset_Button : track 55.9 -> 45.5 mm
- net Y_Button: track 66.1 -> 57.3 mm, vias 4 -> 2
- net DIODE_CLK: track 42.2 -> 49.2 mm
- net Net-(#FLG02-pwr): track 33.8 -> 40.8 mm
- net SWDIO: track 115.7 -> 121.1 mm
- net Li-ion: track 52.4 -> 49.4 mm
- net NES/SNES_switcher: track 35.9 -> 38.9 mm
- net DIODE_OE: track 52.7 -> 55.5 mm, vias 5 -> 4
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