File: Hardware/Kicad/Controller_NRF24L01_Include/Controller_NRF24L01_Include.kicad_pcb (KiCad board)
At the start: 2 copper layers, 90 parts, among them J1 Conn_01x02, J2 Conn_02x07_Odd_Even, SW1 SW_DIP_x01, SW10 SW_DIP_x01, SW11 SW_SPST, SW12 SW_SPST, SW13 SW_SPST, SW2 SW_SPST, SW3 SW_SPST, SW4 SW_SPST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

Commit message: Exculde finish
Parts:
- moved R5 0.17 mm to (185.0, 69.0)
Routing:
- net GND: track 64.7 -> 95.2 mm, vias 4 -> 25
- net Glob_Alim: track 150.5 -> 153.9 mm
- net DIODE_CLK: track 49.2 -> 51.0 mm
- net L: track 117.6 -> 118.7 mm
- net USART2_RX: track 30.1 -> 30.7 mm
