File: Hardware/Kicad/Controller_NRF24L01_Include/Controller_NRF24L01_Include.kicad_sch (KiCad schematic)
At the start: 67 parts, among them J1 Conn_01x02, SW1 SW_Push, SW10 SW_Push, SW11 SW_DIP_x01, SW12 SW_Push, SW13 SW_DIP_x01, SW2 SW_Push, SW3 SW_Push, SW4 SW_Push, SW5 SW_Push, SW6 SW_Push, SW7 SW_Push, SW8 SW_Push, SW9 SW_Push, U1 STM32L412KBTx, U2 MIC5219-3.3YMM, U3 NRF24L01, Y1 16MHz

Commit message: L ET RRRRRRRRRRRRRRRRRRRRRR
Parts:
- Y1: footprint Oscillator:Oscillator_SMD_EuroQuartz_XO91-4Pin_7.0x5.0mm -> Crystal:Crystal_SMD_HC49-SD_HandSoldering
Changed lines of the file:
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@@
+    (stroke (width 0) (type default))
+  )
+  (polyline (pts (xy 208.28 120.65) (xy 208.28 165.1))
     (stroke (width 0) (type default))
   )
@@
     (stroke (width 0) (type default))
   )
+  (polyline (pts (xy 208.28 120.65) (xy 241.3 120.65))
+    (stroke (width 0) (type default))
+  )
   (wire (pts (xy 118.11 88.9) (xy 118.11 93.98))
     (stroke (width 0) (type default))
   )
+  (polyline (pts (xy 241.3 165.1) (xy 241.3 120.65))
+    (stroke (width 0) (type default))
+  )
   (wire (pts (xy 185.42 41.91) (xy 185.42 39.37))
     (stroke (width 0) (type default))
@@
   )
   (wire (pts (xy 257.81 99.06) (xy 257.81 102.87))
+    (stroke (width 0) (type default))
+  )
+  (polyline (pts (xy 208.28 165.1) (xy 241.3 165.1))
     (stroke (width 0) (type default))
   )
@@
       (effects (font (size 1.27 1.27)) (justify right))
     )
-    (property "Footprint" "Oscillator:Oscillator_SMD_EuroQuartz_XO91-4Pin_7.0x5.0mm" (at 93.98 170.18 0)
-      (effects (font (size 1.27 1.27)) hide)
-    )
+    (property "Footprint" "Crystal:Crystal_SMD_HC49-SD_HandSoldering" (at 93.98 170.18 0)
+      (effects (font (size 1.27 1.27)) hide)
+    )

Commit message: Thanks M.Papazoglou,more led, more Software problem
Parts:
- removed C12: 1nF, Capacitor_SMD:C_0603_1608Metric_Pad1.08x0.95mm_HandSolder, symbol Device:C_Small
- removed D2, D3, D4, D5, D6: LED, LED_SMD:LED_0603_1608Metric_Pad1.05x0.95mm_HandSolder, symbol Device:LED
- removed R1, R10, R13, R18, R2, R3, R4, R5, R6, R7, R8, R9: 1K, Resistor_SMD:R_0603_1608Metric_Pad0.98x0.95mm_HandSolder, symbol Device:R_Small
- removed R14, R15, R16, R17: R_Small, Resistor_SMD:R_0603_1608Metric_Pad0.98x0.95mm_HandSolder, symbol Device:R_Small
- removed SW1, SW10, SW12, SW2, SW3, SW4, SW5, SW6, SW7, SW8, SW9: SW_Push, Button_Switch_THT:SW_PUSH_6mm_H5mm, symbol Switch:SW_Push
- added J2: Conn_02x07_Odd_Even, Connector_PinHeader_1.27mm:PinHeader_2x07_P1.27mm_Vertical_SMD, symbol Connector_Generic:Conn_02x07_Odd_Even
- added R20, R21: 1K, Resistor_SMD:R_0603_1608Metric_Pad0.98x0.95mm_HandSolder, symbol Device:R_Small
- added SW1, SW10, SW12, SW2, SW3, SW4, SW5, SW6, SW7, SW8, SW9: SW_SPST, Button_Switch_SMD:SW_SPST_B3S-1000, symbol Switch:SW_SPST
- added TP1: R, Connector_Coaxial:SMA_Molex_73251-1153_EdgeMount_Horizontal, symbol Connector:CoaxialSwitch_Testpoint
- added TP2: L, Connector_Coaxial:SMA_Molex_73251-1153_EdgeMount_Horizontal, symbol Connector:CoaxialSwitch_Testpoint
- C2: value 4.7nF -> 4.7pF; footprint Capacitor_SMD:C_0603_1608Metric_Pad1.08x0.95mm_HandSolder -> Capacitor_SMD:C_0402_1005Metric_Pad0.74x0.62mm_HandSolder
- C3: footprint Capacitor_SMD:C_0603_1608Metric_Pad1.08x0.95mm_HandSolder -> Capacitor_SMD:C_0402_1005Metric_Pad0.74x0.62mm_HandSolder
- C4: value 1.5nF -> 1.5pF; footprint Capacitor_SMD:C_0603_1608Metric_Pad1.08x0.95mm_HandSolder -> Capacitor_SMD:C_0402_1005Metric_Pad0.74x0.62mm_HandSolder
- C5: value 1.0nF -> 1.0pF; footprint Capacitor_SMD:C_0603_1608Metric_Pad1.08x0.95mm_HandSolder -> Capacitor_SMD:C_0402_1005Metric_Pad0.74x0.62mm_HandSolder
- L2: value 2.7nF -> 2.7nH; footprint Inductor_SMD:L_0603_1608Metric_Pad1.05x0.95mm_HandSolder -> Inductor_SMD:L_0402_1005Metric_Pad0.77x0.64mm_HandSolder
- L3: value 8.2nF -> 8.2nH
Connections:
- net A_Button: now also SW1.2 (B)
- net B_Button: now also SW2.2 (B)
- net DC_Button: now also SW8.2 (B)
- net GND: now also J2.11 (Pin_11), J2.5 (Pin_5), J2.7 (Pin_7), R20.2, R21.2, SW1.1 (A), SW10.1 (A), SW12.1 (A), SW2.1 (A), SW3.1 (A), SW4.1 (A), SW5.1 (A), SW6.1 (A), SW7.1 (A), SW8.1 (A), SW9.1 (A), TP1.G, TP2.G
- net Glob_Alim: now also TP1.C, TP2.C
- net LC_Button: now also SW6.2 (B)
- net NES/SNES_switcher: now also U1.15 (PB1); no longer U1.23 (PA13)
- net Order_Search: now also SW10.2 (B)
- net RC_Button: now also SW7.2 (B)
- net SE_Button: now also SW12.2 (B)
- net ST_Button: now also SW9.2 (B)
- net UC_Button: now also SW5.2 (B)
- net X_Button: now also U1.3 (PC15), SW3.2 (B); no longer U1.8 (PA2)
- net Y_Button: now also U1.2 (PC14), SW4.2 (B); no longer U1.9 (PA3)
- net POWER_CHECK: now reaches U1.14 (PB0)
- net SWDCK: now reaches U1.24 (PA14)
- net SWDCK: now also J2.6 (Pin_6)
- net DIODE_SDA: now reaches U1.25 (PA15)
- net R: now reaches U1.29 (PB6)
- net R: now also R20.1, TP1.A
- net L: now reaches U1.30 (PB7)
- net L: now also R21.1, TP2.A
- net Reset_Buton : now reaches U1.4 (NRST)
- net Reset_Buton : now also J2.12 (Pin_12)
- net LED_Order: no longer names the net of U1.22 (PA12)
- new net +3.3V: J2.3 (Pin_3)
- new net SWDIO: J2.4 (Pin_4), U1.23 (PA13)
- new net USART2_RX: J2.13 (Pin_13), U1.9 (PA3)
- new net USART2_TX: J2.14 (Pin_14), U1.8 (PA2)
- no-connect marks 13 -> 10
Other:
- added sheet DIODE (DIODE_sch.kicad_sch)
- note added: "L/R switcher"
- note added: "SWD Connector"
- note added: "SWITCH NES/SNES"
- note removed: "ENERGY LEVEL"
- moved on the sheet: D7, U1

Commit message: New controler versions, and not the last
Parts:
- renumbered C10 to C1, C1 to C10, C3 to C11, C2 to C12, C8 to C2, C9 to C3, C13 to C4, C4 to C5, C5 to C6, C6 to C7, C7 to C8, C11 to C9, D7 to D1, D1 to D2, L3 to L1, L1 to L2, L2 to L3, R12 to R1, R11 to R2, R19 to R3, R20 to R4, R21 to R5, SW11 to SW1, SW13 to SW10, SW8 to SW11, SW9 to SW12, SW12 to SW13, SW1 to SW2, SW2 to SW3, SW3 to SW4, SW4 to SW5, SW5 to SW6, SW10 to SW7, SW6 to SW8, SW7 to SW9, U3 to U2, U2 to U3
Connections:
- net DC_Button: now also U1.27 (PB4); no longer U1.11 (PA5)
- net DIODE_SDA: now also U1.22 (PA12); no longer U1.25 (PA15)
- net Digital_Out_Put: now also U1.12 (PA6); no longer U1.27 (PB4)
- net LC_Button: now also U1.26 (PB3); no longer U1.12 (PA6)
- net MOSI: now also U1.13 (PA7); no longer U1.28 (PB5)
- net NES/SNES_switcher: now also U1.31 (PH3); no longer U1.15 (PB1)
- net Order_Search: now also U1.10 (PA4); no longer U1.20 (PA10)
- net Pin_Clock: now also U1.11 (PA5); no longer U1.26 (PB3)
- net RC_Button: now also U1.15 (PB1); no longer U1.13 (PA7)
- net UC_Button: now also U1.28 (PB5); no longer U1.10 (PA4)
- new net DIODE_CLK: U1.20 (PA10)
- new net DIODE_OE: U1.25 (PA15)
- no-connect marks 10 -> 8
Other:
- moved on the sheet: D1, U1

Commit message: New New controler vers
Changed lines of the file:
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@@
   (junction (at 125.73 53.34) (diameter 0) (color 0 0 0 0)
   )
+  (junction (at 242.57 140.97) (diameter 0) (color 0 0 0 0)
+  )
   (junction (at 72.39 182.88) (diameter 0) (color 0 0 0 0)
   )
@@
   )
   (junction (at 109.22 78.74) (diameter 0) (color 0 0 0 0)
-  )
-  (junction (at 246.38 139.7) (diameter 0) (color 0 0 0 0)
   )
   (junction (at 160.02 147.32) (diameter 0) (color 0 0 0 0)
@@
     (stroke (width 0) (type default))
   )
-  (wire (pts (xy 246.38 140.97) (xy 246.38 139.7))
-    (stroke (width 0) (type default))
-  )
   (wire (pts (xy 91.44 73.66) (xy 91.44 78.74))
     (stroke (width 0) (type default))
@@
     (stroke (width 0) (type default))
   )
-  (wire (pts (xy 252.73 140.97) (xy 246.38 140.97))
-    (stroke (width 0) (type default))
-  )
   (wire (pts (xy 227.33 129.54) (xy 227.33 138.43))
     (stroke (width 0) (type default))
@@
     (stroke (width 0) (type default))
   )
+  (wire (pts (xy 242.57 140.97) (xy 252.73 140.97))
+    (stroke (width 0) (type default))
+  )
   (polyline (pts (xy 87.63 62.23) (xy 157.48 62.23))
     (stroke (width 0) (type default))
@@
   )
   (wire (pts (xy 257.81 78.74) (xy 257.81 83.82))
+    (stroke (width 0) (type default))
+  )
+  (wire (pts (xy 240.03 140.97) (xy 242.57 140.97))
     (stroke (width 0) (type default))
   )
@@
     )
   )
-  (symbol (lib_id "power:+3.3V") (at 246.38 139.7 0) (unit 1)
-    (in_bom yes) (on_board yes) (dnp no) (fields_autoplaced)
-    (property "Reference" "#PWR020" (at 246.38 143.51 0)
-      (effects (font (size 1.27 1.27)) hide)
-    )
-    (property "Value" "+3.3V" (at 246.38 135.89 0)
-      (effects (font (size 1.27 1.27)))
-    )
-    (property "Footprint" "" (at 246.38 139.7 0)
-      (effects (font (size 1.27 1.27)) hide)
-    )
-    (property "Datasheet" "" (at 246.38 139.7 0)
-      (effects (font (size 1.27 1.27)) hide)
-    )
-    (pin "1")
-    (instances
-      (project "Controller_NRF24L01_Include"
-        (path "/700f508b-c905-4d29-9c95-836d8db731fc"
-          (reference "#PWR020") (unit 1)
-        )
-      )
-      (project "Controler_NRF24L01_Exclude"
-        (path "/76ef48f1-60b7-4c4b-a0ce-73b6af33b115"
-          (reference "#PWR?") (unit 1)
-        )
-      )
-      (project "PCBschematic"
-        (path "/cc300af8-7dc6-4303-a7a3-6c9320b23fa8"
-          (reference "#PWR?") (unit 1)
+  (symbol (lib_id "power:PWR_FLAG") (at 242.57 140.97 0) (unit 1)
+    (in_bom yes) (on_board yes) (dnp no)
+    (property "Reference" "#FLG07" (at 242.57 139.065 0)
+      (effects (font (size 1.27 1.27)) hide)
+    )
+    (property "Value" "PWR_FLAG" (at 248.92 139.7 0)
+      (effects (font (size 1.27 1.27)))
+    )
+    (property "Footprint" "" (at 242.57 140.97 0)
+      (effects (font (size 1.27 1.27)) hide)
+    )
+    (property "Datasheet" "~" (at 242.57 140.97 0)
+      (effects (font (size 1.27 1.27)) hide)
+    )
+    (pin "1")
+    (instances
+      (project "Controller_NRF24L01_Include"
+        (path "/700f508b-c905-4d29-9c95-836d8db731fc"
+          (reference "#FLG07") (unit 1)
         )
       )
@@
         (path "/700f508b-c905-4d29-9c95-836d8db731fc"
           (reference "R4") (unit 1)
-        )
-      )
-    )
-  )
-  (symbol (lib_id "power:+3.3V") (at 246.38 139.7 0) (unit 1)
-    (in_bom yes) (on_board yes) (dnp no) (fields_autoplaced)
-    (property "Reference" "#PWR021" (at 246.38 143.51 0)
-      (effects (font (size 1.27 1.27)) hide)
-    )
-    (property "Value" "+3.3V" (at 246.38 135.89 0)
-      (effects (font (size 1.27 1.27)))
-    )
-    (property "Footprint" "" (at 246.38 139.7 0)
-      (effects (font (size 1.27 1.27)) hide)
-    )
-    (property "Datasheet" "" (at 246.38 139.7 0)
-      (effects (font (size 1.27 1.27)) hide)
-    )
-    (pin "1")
-    (instances
-      (project "Controller_NRF24L01_Include"
-        (path "/700f508b-c905-4d29-9c95-836d8db731fc"
-          (reference "#PWR021") (unit 1)
-        )
-      )
-      (project "Controler_NRF24L01_Exclude"
-        (path "/76ef48f1-60b7-4c4b-a0ce-73b6af33b115"
-          (reference "#PWR?") (unit 1)
-        )
-      )
-      (project "PCBschematic"
-        (path "/cc300af8-7dc6-4303-a7a3-6c9320b23fa8"
-          (reference "#PWR?") (unit 1)
         )
       )
@@
         )
       )
+    )
+  )
+  (symbol (lib_id "power:+3.3V") (at 240.03 140.97 0) (unit 1)
+    (in_bom yes) (on_board yes) (dnp no) (fields_autoplaced)
+    (property "Reference" "#PWR020" (at 240.03 144.78 0)
+      (effects (font (size 1.27 1.27)) hide)
+    )
+    (property "Value" "+3.3V" (at 240.03 137.16 0)
+      (effects (font (size 1.27 1.27)))
+    )
+    (property "Footprint" "" (at 240.03 140.97 0)
+      (effects (font (size 1.27 1.27)) hide)
+    )
+    (property "Datasheet" "" (at 240.03 140.97 0)
+      (effects (font (size 1.27 1.27)) hide)
+    )
+    (pin "1")
+    (instances
+      (project "Controller_NRF24L01_Include"
+        (path "/700f508b-c905-4d29-9c95-836d8db731fc"
+          (reference "#PWR020") (unit 1)
+        )
+      )

Commit message: And a new version of the controler
Changed lines of the file:
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@@
+    (stroke (width 0) (type default))
+  )
+  (wire (pts (xy 151.13 176.53) (xy 157.48 176.53))
     (stroke (width 0) (type default))
   )
@@
     (stroke (width 0) (type default))
   )
+  (wire (pts (xy 146.05 182.88) (xy 157.48 182.88))
+    (stroke (width 0) (type default))
+  )
   (wire (pts (xy 209.55 132.08) (xy 209.55 138.43))
     (stroke (width 0) (type default))
@@
   )
   (wire (pts (xy 156.21 147.32) (xy 160.02 147.32))
-    (stroke (width 0) (type default))
-  )
-  (wire (pts (xy 151.13 182.88) (xy 157.48 182.88))
     (stroke (width 0) (type default))
   )
@@
     )
   )
-  (global_label "Antenna" (shape input) (at 157.48 176.53 180) (fields_autoplaced)
-    (effects (font (size 1.27 1.27)) (justify right))
-    (property "Intersheetrefs" "${INTERSHEET_REFS}" (at 147.0753 176.53 0)
+  (global_label "Antenna" (shape input) (at 151.13 176.53 180) (fields_autoplaced)
+    (effects (font (size 1.27 1.27)) (justify right))
+    (property "Intersheetrefs" "${INTERSHEET_REFS}" (at 140.7253 176.53 0)
       (effects (font (size 1.27 1.27)) (justify right) hide)
     )
@@
     )
   )
-  (netclass_flag "" (length 2.54) (shape round) (at 151.13 182.88 0) (fields_autoplaced)
+  (netclass_flag "" (length 2.54) (shape round) (at 146.05 182.88 0) (fields_autoplaced)
     (effects (font (size 1.27 1.27)) (justify left bottom))
-    (property "Netclass" "Antenna" (at 151.8285 180.34 0)
+    (property "Netclass" "Antenna" (at 146.7485 180.34 0)
       (effects (font (size 1.27 1.27) italic) (justify left) hide)
     )
@@
     )
   )
-  (symbol (lib_id "power:GND") (at 151.13 182.88 0) (unit 1)
-    (in_bom yes) (on_board yes) (dnp no) (fields_autoplaced)
-    (property "Reference" "#PWR09" (at 151.13 189.23 0)
-      (effects (font (size 1.27 1.27)) hide)
-    )
-    (property "Value" "GND" (at 151.13 187.96 0)
-      (effects (font (size 1.27 1.27)))
-    )
-    (property "Footprint" "" (at 151.13 182.88 0)
-      (effects (font (size 1.27 1.27)) hide)
-    )
-    (property "Datasheet" "" (at 151.13 182.88 0)
-      (effects (font (size 1.27 1.27)) hide)
-    )
+  (symbol (lib_id "power:GND") (at 146.05 182.88 0) (unit 1)
+    (in_bom yes) (on_board yes) (dnp no) (fields_autoplaced)
+    (property "Reference" "#PWR09" (at 146.05 189.23 0)
+      (effects (font (size 1.27 1.27)) hide)
+    )
+    (property "Value" "GND" (at 146.05 187.96 0)
+      (effects (font (size 1.27 1.27)))
+    )
+    (property "Footprint" "" (at 146.05 182.88 0)
+      (effects (font (size 1.27 1.27)) hide)
+    )
+    (property "Datasheet" "" (at 146.05 182.88 0)
+      (effects (font (size 1.27 1.27)) hide)
+    )

Commit message: Maybe the final version
Connections:
- net DC_Button: now also U1.14 (PB0); no longer U1.27 (PB4)
- net DIODE_CLK: now also U1.26 (PB3); no longer U1.20 (PA10)
- net DIODE_SDA: now also U1.28 (PB5); no longer U1.22 (PA12)
- net LC_Button: now also U1.3 (PC15); no longer U1.26 (PB3)
- net POWER_CHECK: now also U1.27 (PB4); no longer U1.14 (PB0)
- net RC_Button: now also U1.2 (PC14); no longer U1.15 (PB1)
- net UC_Button: now also U1.15 (PB1); no longer U1.28 (PB5)
- net X_Button: now also U1.20 (PA10); no longer U1.3 (PC15)
- net Y_Button: now also U1.22 (PA12); no longer U1.2 (PC14)
- net Reset_Buton  renamed Reset_Button 
Changed lines of the file:
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@@
     )
   )
-  (global_label "DC_Button" (shape input) (at 40.64 74.93 180) (fields_autoplaced)
-    (effects (font (size 1.27 1.27)) (justify right))
-    (property "Intersheetrefs" "${INTERSHEET_REFS}" (at 28.0582 74.93 0)
+  (global_label "DC_Button" (shape input) (at 40.64 67.31 180) (fields_autoplaced)
+    (effects (font (size 1.27 1.27)) (justify right))
+    (property "Intersheetrefs" "${INTERSHEET_REFS}" (at 28.0582 67.31 0)
       (effects (font (size 1.27 1.27)) (justify right) hide)
     )
@@
     )
   )
-  (global_label "LC_Button" (shape input) (at 40.64 72.39 180) (fields_autoplaced)
-    (effects (font (size 1.27 1.27)) (justify right))
-    (property "Intersheetrefs" "${INTERSHEET_REFS}" (at 28.3001 72.39 0)
-      (effects (font (size 1.27 1.27)) (justify right) hide)
-    )
-  )
-  (global_label "DIODE_CLK" (shape input) (at 66.04 74.93 0) (fields_autoplaced)
-    (effects (font (size 1.27 1.27)) (justify left))
-    (property "Intersheetrefs" "${INTERSHEET_REFS}" (at 79.1058 74.93 0)
-      (effects (font (size 1.27 1.27)) (justify left) hide)
+  (global_label "LC_Button" (shape input) (at 40.64 62.23 180) (fields_autoplaced)
+    (effects (font (size 1.27 1.27)) (justify right))
+    (property "Intersheetrefs" "${INTERSHEET_REFS}" (at 28.3001 62.23 0)
+      (effects (font (size 1.27 1.27)) (justify right) hide)
+    )
+  )
+  (global_label "DIODE_CLK" (shape input) (at 40.64 72.39 180) (fields_autoplaced)
+    (effects (font (size 1.27 1.27)) (justify right))
+    (property "Intersheetrefs" "${INTERSHEET_REFS}" (at 27.5742 72.39 0)
+      (effects (font (size 1.27 1.27)) (justify right) hide)
     )
   )
@@
     )
   )
-  (global_label "Y_Button" (shape input) (at 40.64 59.69 180) (fields_autoplaced)
-    (effects (font (size 1.27 1.27)) (justify right))
-    (property "Intersheetrefs" "${INTERSHEET_REFS}" (at 29.5096 59.69 0)
-      (effects (font (size 1.27 1.27)) (justify right) hide)
-    )
-  )
-  (global_label "Reset_Buton " (shape input) (at 40.64 49.53 180) (fields_autoplaced)
-    (effects (font (size 1.27 1.27)) (justify right))
-    (property "Intersheetrefs" "${INTERSHEET_REFS}" (at 25.3609 49.53 0)
-      (effects (font (size 1.27 1.27)) (justify right) hide)
-    )
-  )
-  (global_label "POWER_CHECK" (shape input) (at 40.64 67.31 180) (fields_autoplaced)
-    (effects (font (size 1.27 1.27)) (justify right))
-    (property "Intersheetrefs" "${INTERSHEET_REFS}" (at 24.0062 67.31 0)
+  (global_label "Y_Button" (shape input) (at 66.04 80.01 0) (fields_autoplaced)
+    (effects (font (size 1.27 1.27)) (justify left))
+    (property "Intersheetrefs" "${INTERSHEET_REFS}" (at 77.1704 80.01 0)
+      (effects (font (size 1.27 1.27)) (justify left) hide)
+    )
+  )
+  (global_label "Reset_Button " (shape input) (at 40.64 49.53 180) (fields_autoplaced)
+    (effects (font (size 1.27 1.27)) (justify right))
+    (property "Intersheetrefs" "${INTERSHEET_REFS}" (at 24.6352 49.53 0)
+      (effects (font (size 1.27 1.27)) (justify right) hide)
+    )
+  )
+  (global_label "POWER_CHECK" (shape input) (at 40.64 74.93 180) (fields_autoplaced)
+    (effects (font (size 1.27 1.27)) (justify right))
+    (property "Intersheetrefs" "${INTERSHEET_REFS}" (at 24.0062 74.93 0)
       (effects (font (size 1.27 1.27)) (justify right) hide)
     )
@@
     )
   )
-  (global_label "UC_Button" (shape input) (at 40.64 77.47 180) (fields_autoplaced)
-    (effects (font (size 1.27 1.27)) (justify right))
-    (property "Intersheetrefs" "${INTERSHEET_REFS}" (at 27.9977 77.47 0)
+  (global_label "UC_Button" (shape input) (at 40.64 69.85 180) (fields_autoplaced)
+    (effects (font (size 1.27 1.27)) (justify right))
+    (property "Intersheetrefs" "${INTERSHEET_REFS}" (at 27.9977 69.85 0)
       (effects (font (size 1.27 1.27)) (justify right) hide)
     )
@@
     )
   )
-  (global_label "Reset_Buton " (shape input) (at 265.43 151.13 0) (fields_autoplaced)
-    (effects (font (size 1.27 1.27)) (justify left))
-    (property "Intersheetrefs" "${INTERSHEET_REFS}" (at 280.7091 151.13 0)
+  (global_label "Reset_Button " (shape input) (at 265.43 151.13 0) (fields_autoplaced)
+    (effects (font (size 1.27 1.27)) (justify left))
+    (property "Intersheetrefs" "${INTERSHEET_REFS}" (at 281.4348 151.13 0)
       (effects (font (size 1.27 1.27)) (justify left) hide)
     )
@@
     )
   )
-  (global_label "X_Button" (shape input) (at 40.64 62.23 180) (fields_autoplaced)
-    (effects (font (size 1.27 1.27)) (justify right))
-    (property "Intersheetrefs" "${INTERSHEET_REFS}" (at 29.3887 62.23 0)
-      (effects (font (size 1.27 1.27)) (justify right) hide)
+  (global_label "X_Button" (shape input) (at 66.04 74.93 0) (fields_autoplaced)
+    (effects (font (size 1.27 1.27)) (justify left))
+    (property "Intersheetrefs" "${INTERSHEET_REFS}" (at 77.2913 74.93 0)
+      (effects (font (size 1.27 1.27)) (justify left) hide)
     )
   )
@@
     )
   )
-  (global_label "RC_Button" (shape input) (at 40.64 69.85 180) (fields_autoplaced)
-    (effects (font (size 1.27 1.27)) (justify right))
-    (property "Intersheetrefs" "${INTERSHEET_REFS}" (at 28.0582 69.85 0)
+  (global_label "RC_Button" (shape input) (at 40.64 59.69 180) (fields_autoplaced)
+    (effects (font (size 1.27 1.27)) (justify right))
+    (property "Intersheetrefs" "${INTERSHEET_REFS}" (at 28.0582 59.69 0)
       (effects (font (size 1.27 1.27)) (justify right) hide)
     )
@@
     )
   )
-  (global_label "DIODE_SDA" (shape input) (at 66.04 80.01 0) (fields_autoplaced)
-    (effects (font (size 1.27 1.27)) (justify left))
-    (property "Intersheetrefs" "${INTERSHEET_REFS}" (at 79.1058 80.01 0)
-      (effects (font (size 1.27 1.27)) (justify left) hide)
-    )
-  )
+  (global_label "DIODE_SDA" (shape input) (at 40.64 77.47 180) (fields_autoplaced)
+    (effects (font (size 1.27 1.27)) (justify right))
+    (property "Intersheetrefs" "${INTERSHEET_REFS}" (at 27.5742 77.47 0)
+      (effects (font (size 1.27 1.27)) (justify right) hide)
+    )
+  )
