File: Hardware/Kicad/Controller_NRF24L01_Include/DIODE_sch.kicad_sch (KiCad schematic)
At the start: 22 parts, among them U4 PCA9685PW

Commit message: New vers Controler
Connections:
- net GND: now also U4.24 (A5), U4.4 (A3), U4.5 (A4)
- net Li-ion: no longer C14.1, D20.2 (A)
- new net Glob_Alim: C14.1, D20.2 (A)
Changed lines of the file:
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@@
   (junction (at 176.53 85.09) (diameter 0) (color 0 0 0 0)
   )
+  (junction (at 158.75 71.12) (diameter 0) (color 0 0 0 0)
+  )
   (junction (at 135.89 40.64) (diameter 0) (color 0 0 0 0)
   )
+  (junction (at 158.75 85.09) (diameter 0) (color 0 0 0 0)
+  )
   (junction (at 251.46 31.75) (diameter 0) (color 0 0 0 0)
   )
@@
   (junction (at 205.74 53.34) (diameter 0) (color 0 0 0 0)
   )
+  (junction (at 158.75 68.58) (diameter 0) (color 0 0 0 0)
+  )
   (junction (at 205.74 50.8) (diameter 0) (color 0 0 0 0)
   )
@@
     (stroke (width 0) (type default))
   )
+  (wire (pts (xy 158.75 85.09) (xy 176.53 85.09))
+    (stroke (width 0) (type default))
+  )
   (wire (pts (xy 242.57 25.4) (xy 251.46 25.4))
     (stroke (width 0) (type default))
@@
     (stroke (width 0) (type default))
   )
+  (wire (pts (xy 158.75 71.12) (xy 158.75 85.09))
+    (stroke (width 0) (type default))
+  )
   (wire (pts (xy 205.74 66.04) (xy 205.74 63.5))
     (stroke (width 0) (type default))
@@
     (stroke (width 0) (type default))
   )
+  (wire (pts (xy 158.75 68.58) (xy 158.75 71.12))
+    (stroke (width 0) (type default))
+  )
   (wire (pts (xy 205.74 86.36) (xy 205.74 85.09))
     (stroke (width 0) (type default))
@@
     (stroke (width 0) (type default))
   )
-  (wire (pts (xy 135.89 85.09) (xy 176.53 85.09))
+  (wire (pts (xy 135.89 85.09) (xy 158.75 85.09))
+    (stroke (width 0) (type default))
+  )
+  (wire (pts (xy 158.75 66.04) (xy 158.75 68.58))
     (stroke (width 0) (type default))
   )
@@
     )
   )
-  (global_label "Li-ion" (shape input) (at 135.89 27.94 180) (fields_autoplaced)
+  (global_label "Glob_Alim" (shape input) (at 135.89 27.94 180) (fields_autoplaced)
     (effects (font (size 1.27 1.27) bold) (justify right))
-    (property "Intersheetrefs" "${INTERSHEET_REFS}" (at 126.4477 26.67 0)
+    (property "Intersheetrefs" "${INTERSHEET_REFS}" (at 123.3031 27.94 0)
       (effects (font (size 1.27 1.27)) (justify right) hide)
     )

Commit message: New controler versions, and not the last
Parts:
- removed C14: 1uF, symbol Device:C_Small
- added R10, R8, R9: 10K, Resistor_SMD:R_0603_1608Metric_Pad0.98x0.95mm_HandSolder, symbol Device:R_Small
- added R11, R12, R13, R14, R15, R16, R17, R18, R19, R20, R21, R22, R23, R24, R25, R26: 1K, Resistor_SMD:R_0603_1608Metric_Pad0.98x0.95mm_HandSolder, symbol Device:R_Small
- D10: value LED -> G7; footprint Display:HDSP-4832 -> LED_SMD:LED_0603_1608Metric_Pad1.05x0.95mm_HandSolder
- D11: value LED -> G8; footprint Display:HDSP-4832 -> LED_SMD:LED_0603_1608Metric_Pad1.05x0.95mm_HandSolder
- D12: value LED -> O1; footprint Display:HDSP-4832 -> LED_SMD:LED_0603_1608Metric_Pad1.05x0.95mm_HandSolder
- D13: value LED -> O2; footprint Display:HDSP-4832 -> LED_SMD:LED_0603_1608Metric_Pad1.05x0.95mm_HandSolder
- D14: value LED -> O3; footprint Display:HDSP-4832 -> LED_SMD:LED_0603_1608Metric_Pad1.05x0.95mm_HandSolder
- D15: value LED -> O4; footprint Display:HDSP-4832 -> LED_SMD:LED_0603_1608Metric_Pad1.05x0.95mm_HandSolder
- D16: value LED -> R1; footprint Display:HDSP-4832 -> LED_SMD:LED_0603_1608Metric_Pad1.05x0.95mm_HandSolder
- D17: value LED -> R2; footprint Display:HDSP-4832 -> LED_SMD:LED_0603_1608Metric_Pad1.05x0.95mm_HandSolder
- D18: value LED -> R3; footprint Display:HDSP-4832 -> LED_SMD:LED_0603_1608Metric_Pad1.05x0.95mm_HandSolder
- D19: value LED -> R4; footprint Display:HDSP-4832 -> LED_SMD:LED_0603_1608Metric_Pad1.05x0.95mm_HandSolder
- D3: renamed from D20; footprint (none) -> Display:HDSP-4832
- D4: renamed from D3; value LED -> G1; footprint Display:HDSP-4832 -> LED_SMD:LED_0603_1608Metric_Pad1.05x0.95mm_HandSolder
- D5: renamed from D4; value LED -> G2; footprint Display:HDSP-4832 -> LED_SMD:LED_0603_1608Metric_Pad1.05x0.95mm_HandSolder
- D6: renamed from D5; value LED -> G3; footprint Display:HDSP-4832 -> LED_SMD:LED_0603_1608Metric_Pad1.05x0.95mm_HandSolder
- D7: renamed from D6; value LED -> G4; footprint Display:HDSP-4832 -> LED_SMD:LED_0603_1608Metric_Pad1.05x0.95mm_HandSolder
- D8: value LED -> G5; footprint Display:HDSP-4832 -> LED_SMD:LED_0603_1608Metric_Pad1.05x0.95mm_HandSolder
- D9: value LED -> G6; footprint Display:HDSP-4832 -> LED_SMD:LED_0603_1608Metric_Pad1.05x0.95mm_HandSolder
- R6: renamed from R1; footprint (none) -> Resistor_SMD:R_0603_1608Metric_Pad0.98x0.95mm_HandSolder
- R7: renamed from R2; footprint (none) -> Resistor_SMD:R_0603_1608Metric_Pad0.98x0.95mm_HandSolder
- renumbered C12 to C?
Connections:
- net DIODE_SDA: now also R8.1
- net GND: now also U4.2 (A1), R11.2, R12.2, R13.2, R14.2, R15.2, R16.2, R17.2, R18.2, R19.2, R20.2, R21.2, R22.2, R23.2, R24.2, R25.2, R26.2; no longer D10.1 (K), D11.1 (K), D12.1 (K), D13.1 (K), D14.1 (K), D15.1 (K), D16.1 (K), D17.1 (K), D18.1 (K), D19.1 (K), D4.1 (K), D5.1 (K), D6.1 (K), D7.1 (K), D8.1 (K), D9.1 (K), U4.5 (A4)
- net Glob_Alim: now also U4.1 (A0), U4.3 (A2), U4.5 (A4), R10.2, R8.2, R9.1
- net DIODE_OE: now reaches U4.23 (~{OE})
- net DIODE_OE: now also R10.1
- net DIODE_CLK: now reaches U4.26 (SCL)
- net DIODE_CLK: now also R9.2
- new net: D11.1 (K), R18.1
- new net: D6.1 (K), R13.1
- new net: D9.1 (K), R16.1
- new net: D19.1 (K), R26.1
- new net: D5.1 (K), R12.1
- new net: D13.1 (K), R20.1
- new net: D7.1 (K), R14.1
- new net: D10.1 (K), R17.1
- new net: D15.1 (K), R22.1
- new net: D8.1 (K), R15.1
- new net: D17.1 (K), R24.1
- new net: D18.1 (K), R25.1
- new net: D12.1 (K), R19.1
- new net: D14.1 (K), R21.1
- new net: D4.1 (K), R11.1
- new net: D16.1 (K), R23.1
Other:
- company: (none) -> ENSEA
- title: (none) -> Diode for Snes controler 
- moved on the sheet: D10, D11, D12, D13, D14, D15, D16, D17, D18, D19, D3, D4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

Commit message: New New controler vers
Parts:
- D3: footprint Display:HDSP-4832 -> LED_SMD:LED_0603_1608Metric_Pad1.05x0.95mm_HandSolder
Changed lines of the file:
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@@
   (junction (at 189.23 29.21) (diameter 0) (color 0 0 0 0)
+  )
+  (junction (at 212.09 29.21) (diameter 0) (color 0 0 0 0)
   )
   (wire (pts (xy 201.93 25.4) (xy 201.93 29.21))
@@
         (path "/700f508b-c905-4d29-9c95-836d8db731fc/efd5fe6b-cfb4-4a93-a48a-8f57d2a0a889"
           (reference "R13") (unit 1)
+        )
+      )
+    )
+  )
+  (symbol (lib_id "power:PWR_FLAG") (at 212.09 29.21 0) (unit 1)
+    (in_bom yes) (on_board yes) (dnp no)
+    (property "Reference" "#FLG06" (at 212.09 27.305 0)
+      (effects (font (size 1.27 1.27)) hide)
+    )
+    (property "Value" "PWR_FLAG" (at 218.44 27.94 0)
+      (effects (font (size 1.27 1.27)))
+    )
+    (property "Footprint" "" (at 212.09 29.21 0)
+      (effects (font (size 1.27 1.27)) hide)
+    )
+    (property "Datasheet" "~" (at 212.09 29.21 0)
+      (effects (font (size 1.27 1.27)) hide)
+    )
+    (pin "1")
+    (instances
+      (project "Controller_NRF24L01_Include"
+        (path "/700f508b-c905-4d29-9c95-836d8db731fc/efd5fe6b-cfb4-4a93-a48a-8f57d2a0a889"
+          (reference "#FLG06") (unit 1)
         )
       )
@@
       (effects (font (size 1.27 1.27)))
     )
-    (property "Footprint" "Display:HDSP-4832" (at 207.01 29.21 90)
-      (effects (font (size 1.27 1.27)) hide)
-    )
+    (property "Footprint" "LED_SMD:LED_0603_1608Metric_Pad1.05x0.95mm_HandSolder" (at 207.01 29.21 90)
+      (effects (font (size 1.27 1.27)) hide)
+    )
