File: Hardware/Kicad/Controler_NRF24L01_Exclude_v2/Diode.kicad_sch (KiCad schematic)
At the start: 39 parts, among them U4 PCA9685PW

Commit message: V.2 controler
Connections:
- net DIODE_CLK renamed DIO/EX_CLK
- net DIODE_SDA renamed DIO/EX_SDA
Changed lines of the file:
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@@
     (stroke (width 0) (type default))
   )
-  (wire (pts (xy 189.23 34.29) (xy 191.77 34.29))
+  (wire (pts (xy 190.5 34.29) (xy 191.77 34.29))
     (stroke (width 0) (type default))
   )
@@
     )
   )
-  (global_label "DIODE_CLK" (shape input) (at 189.23 34.29 180) (fields_autoplaced)
+  (global_label "DIO{slash}EX_CLK" (shape input) (at 190.5 34.29 180) (fields_autoplaced)
     (effects (font (size 1.27 1.27)) (justify right))
     (property "Intersheetrefs" "${INTERSHEET_REFS}" (at 176.1642 34.29 0)
@@
     )
   )
-  (global_label "DIODE_SDA" (shape input) (at 173.99 41.91 180) (fields_autoplaced)
+  (global_label "DIO{slash}EX_SDA" (shape input) (at 173.99 41.91 180) (fields_autoplaced)
     (effects (font (size 1.27 1.27)) (justify right))
-    (property "Intersheetrefs" "${INTERSHEET_REFS}" (at 160.9242 41.91 0)
+    (property "Intersheetrefs" "${INTERSHEET_REFS}" (at 159.6542 41.91 0)
       (effects (font (size 1.27 1.27)) (justify right) hide)
     )
