File: Hardware/Kicad/Controler_NRF24L01_Exclude_v2/GPIO_extender_sch.kicad_sch (KiCad schematic)
At the start: 0 parts

Commit message: V-1.5 controler
Parts:
- added C7: 100µF, Capacitor_SMD:C_0603_1608Metric_Pad1.08x0.95mm_HandSolder, symbol Device:C_Small
- added R4: 10k, Resistor_SMD:R_0603_1608Metric_Pad0.98x0.95mm_HandSolder, symbol Device:R_Small
- added R5, R6: 1K, Resistor_SMD:R_0603_1608Metric_Pad0.98x0.95mm_HandSolder, symbol Device:R_Small
- added U5: PCF8574TS, Package_SO:SSOP-20_4.4x6.5mm_P0.65mm, symbol Interface_Expansion:PCF8574TS
Connections:
- new net: C7.1, R4.1
- new net DIODE_OE: U5.12 (P2)
- new net GND: R4.2, U5.1 (~{INT}), U5.15 (VSS), U5.6 (A0), U5.7 (A1), U5.9 (A2)
- new net GPIO_EX_CLK: R5.2, U5.2 (SCL)
- new net GPIO_EX_SERIAL_DATA: R6.2, U5.4 (SDA)
- new net Glob_Alim: C7.2, R5.1, R6.1, U5.5 (VDD)
- new net ST_Button: U5.11 (P1)
- new net Y_Button: U5.10 (P0)
- no-connect marks 0 -> 5
Other:
- note added: "GPIO EXTENDER"

Commit message: V.2 controler
Parts:
- R5, R6: value 1K -> 10K
Connections:
- net ST_Button: now also U5.20 (P7); no longer U5.11 (P1)
- net DIODE_OE: no longer names the net of U5.12 (P2)
- net GPIO_EX_CLK renamed DIO/EX_CLK
- net GPIO_EX_SERIAL_DATA renamed DIO/EX_SDA
- net Y_Button: no longer names the net of U5.10 (P0)
- no-connect marks 5 -> 7
Changed lines of the file:
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@@
   (no_connect (at 250.19 59.69))
   (no_connect (at 250.19 64.77))
+  (no_connect (at 250.19 49.53))
   (no_connect (at 250.19 62.23))
-  (no_connect (at 250.19 67.31))
+  (no_connect (at 250.19 52.07))
+  (no_connect (at 250.19 54.61))
   (wire (pts (xy 218.44 62.23) (xy 224.79 62.23))
     (stroke (width 0) (type default))
@@
     )
   )
-  (global_label "GPIO_EX_CLK" (shape input) (at 224.79 49.53 180) (fields_autoplaced)
+  (global_label "DIO{slash}EX_SDA" (shape input) (at 201.93 54.61 0) (fields_autoplaced)
+    (effects (font (size 1.27 1.27)) (justify left))
+    (property "Intersheetrefs" "${INTERSHEET_REFS}" (at 216.2658 54.61 0)
+      (effects (font (size 1.27 1.27)) (justify left) hide)
+    )
+  )
+  (global_label "DIO{slash}EX_CLK" (shape input) (at 224.79 49.53 180) (fields_autoplaced)
     (effects (font (size 1.27 1.27)) (justify right))
-    (property "Intersheetrefs" "${INTERSHEET_REFS}" (at 209.5471 49.53 0)
+    (property "Intersheetrefs" "${INTERSHEET_REFS}" (at 210.4542 49.53 0)
       (effects (font (size 1.27 1.27)) (justify right) hide)
     )
   )
-  (global_label "Y_Button" (shape input) (at 250.19 49.53 0) (fields_autoplaced)
+  (global_label "ST_Button" (shape input) (at 250.19 67.31 0) (fields_autoplaced)
     (effects (font (size 1.27 1.27)) (justify left))
-    (property "Intersheetrefs" "${INTERSHEET_REFS}" (at 261.3204 49.53 0)
-      (effects (font (size 1.27 1.27)) (justify left) hide)
-    )
-  )
-  (global_label "GPIO_EX_SERIAL_DATA" (shape input) (at 201.93 54.61 0) (fields_autoplaced)
-    (effects (font (size 1.27 1.27)) (justify left))
-    (property "Intersheetrefs" "${INTERSHEET_REFS}" (at 225.3372 54.61 0)
-      (effects (font (size 1.27 1.27)) (justify left) hide)
-    )
-  )
-  (global_label "DIODE_OE" (shape input) (at 250.19 54.61 0) (fields_autoplaced)
-    (effects (font (size 1.27 1.27)) (justify left))
-    (property "Intersheetrefs" "${INTERSHEET_REFS}" (at 262.1672 54.61 0)
-      (effects (font (size 1.27 1.27)) (justify left) hide)
-    )
-  )
-  (global_label "ST_Button" (shape input) (at 250.19 52.07 0) (fields_autoplaced)
-    (effects (font (size 1.27 1.27)) (justify left))
-    (property "Intersheetrefs" "${INTERSHEET_REFS}" (at 262.4089 52.07 0)
+    (property "Intersheetrefs" "${INTERSHEET_REFS}" (at 262.4089 67.31 0)
       (effects (font (size 1.27 1.27)) (justify left) hide)
     )
@@
       (effects (font (size 1.27 1.27)) (justify left))
     )
-    (property "Value" "1K" (at 212.09 33.655 0)
+    (property "Value" "10K" (at 212.09 33.655 0)
       (effects (font (size 1.27 1.27)) (justify left))
     )
@@
       (effects (font (size 1.27 1.27)) (justify left))
     )
-    (property "Value" "1K" (at 228.6 33.655 0)
-      (effects (font (size 1.27 1.27)) (justify left))
-    )
+    (property "Value" "10K" (at 228.6 33.655 0)
+      (effects (font (size 1.27 1.27)) (justify left))
+    )
