File: Hardware/Kicad/Controler_NRF24L01_Exclude_v2/Controler_NRF24L01_Exclude_v2.kicad_pcb (KiCad board)
At the start: 2 copper layers, 160.2 x 60.2 mm, 77 parts, among them J1 Conn_01x02, J2 Conn_02x07_Odd_Even, J3 Conn_01x03, J4 Conn_01x03, SW1 SW_DIP_x01, SW10 SW_DIP_x01, SW11 SW_Push, SW12 SW_Push, SW13 SW_Push, SW2 SW_Push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

Commit message: V-1.5 controler
Parts:
- added C7: 100µF, Capacitor_SMD:C_0603_1608Metric_Pad1.08x0.95mm_HandSolder, F.Cu at (138.0, 90.2)
- added R4: 10k, Resistor_SMD:R_0603_1608Metric_Pad0.98x0.95mm_HandSolder, F.Cu at (142.4, 88.9)
- added R5: 1K, Resistor_SMD:R_0603_1608Metric_Pad0.98x0.95mm_HandSolder, F.Cu at (130.2, 54.4)
- added R6: 1K, Resistor_SMD:R_0603_1608Metric_Pad0.98x0.95mm_HandSolder, F.Cu at (124.5, 54.4)
- added U5: PCF8574TS, Package_SO:SSOP-20_4.4x6.5mm_P0.65mm, F.Cu at (136.1, 84.9)
- C1: footprint Capacitor_SMD:CP_Elec_5x5.4 -> Capacitor_SMD:C_0603_1608Metric_Pad1.08x0.95mm_HandSolder; moved to B.Cu
- C3, C5, C6: footprint Resistor_SMD:R_0603_1608Metric_Pad0.98x0.95mm_HandSolder -> Capacitor_SMD:C_0603_1608Metric_Pad1.08x0.95mm_HandSolder
- R3: value R_Small -> 1K
- moved C1 3.36 mm to (138.4, 61.9)
Connections:
- U1 pad 18: Y_Button -> GPIO_EX_CLK
- U1 pad 22: ST_Button -> GPIO_EX_SERIAL_DATA
- U1 pad 25: unconnected-(U1-PA15-Pad25) -> CSN_nRF24
- U2 pad 4: unconnected-(U2-CSN-Pad4) -> CSN_nRF24
Routing:
- net CSN_nRF24: track 0.00 -> 69.3 mm, vias 0 -> 1
- net DIODE_OE: track 7.14 -> 28.8 mm, vias 0 -> 2
- net ST_Button: track 18.4 -> 30.4 mm, vias 0 -> 2
- net GPIO_EX_CLK: track 0.00 -> 8.79 mm, vias 0 -> 2
- net GPIO_EX_SERIAL_DATA: track 0.00 -> 7.89 mm, vias 0 -> 2
- net RX/TX: track 35.5 -> 39.6 mm
- net GND: track 23.1 -> 27.2 mm
- net R: track 69.7 -> 73.4 mm
- net Net-(C7-Pad1): track 0.00 -> 3.70 mm
- net Y_Button: track 55.3 -> 53.6 mm
- net NES/SNES_switcher: track 27.1 -> 26.4 mm

Commit message: V.2 controler
Parts:
- R5, R6: value 1K -> 10K
- moved R5 38.4 mm to (137.2, 92.2), turned to 180 degrees
- moved R6 38.2 mm to (136.6, 90.6), turned to 180 degrees
- moved C7 2.00 mm to (140.0, 90.2)
- moved J1 0.88 mm to (177.3, 108.4)
Connections:
- R11 pad 1: DIODE_SDA -> DIO/EX_SDA
- R14 pad 2: DIODE_CLK -> DIO/EX_CLK
- R5 pad 2: GPIO_EX_CLK -> DIO/EX_CLK
- R6 pad 2: GPIO_EX_SERIAL_DATA -> DIO/EX_SDA
- U1 pad 18: GPIO_EX_CLK -> R
- U1 pad 19: NES/SNES_switcher -> DIO/EX_CLK
- U1 pad 20: R -> DIO/EX_SDA
- U1 pad 22: GPIO_EX_SERIAL_DATA -> Y_Button
- U1 pad 26: DIODE_CLK -> DIODE_OE
- U1 pad 28: DIODE_SDA -> NES/SNES_switcher
- U4 pad 26: DIODE_CLK -> DIO/EX_CLK
- U4 pad 27: DIODE_SDA -> DIO/EX_SDA
- U5 pad 10: Y_Button -> unconnected-(U5-P0-Pad10)
- U5 pad 11: ST_Button -> unconnected-(U5-P1-Pad11)
- U5 pad 12: DIODE_OE -> unconnected-(U5-P2-Pad12)
- U5 pad 2: GPIO_EX_CLK -> DIO/EX_CLK
- U5 pad 20: unconnected-(U5-P7-Pad20) -> ST_Button
- U5 pad 4: GPIO_EX_SERIAL_DATA -> DIO/EX_SDA
Routing:
- net DIODE_SDA: track 49.0 -> 0.00 mm, vias 2 -> 0
- net DIODE_CLK: track 48.2 -> 0.00 mm, vias 2 -> 0
- net DIO/EX_SDA: track 0.00 -> 45.2 mm, vias 0 -> 2
- net DIO/EX_CLK: track 0.00 -> 45.0 mm, vias 0 -> 4
- net DIODE_OE: track 28.8 -> 59.0 mm
- net GND: track 27.2 -> 47.4 mm, vias 60 -> 63
- net GPIO_EX_CLK: track 8.79 -> 0.00 mm, vias 2 -> 0
- net GPIO_EX_SERIAL_DATA: track 7.89 -> 0.00 mm, vias 2 -> 0
- net ST_Button: track 30.4 -> 24.5 mm
- net Glob_Alim: track 252.5 -> 258.0 mm
- net Y_Button: track 53.6 -> 55.6 mm
- net Net-(C7-Pad1): track 3.70 -> 2.19 mm
- net R: track 73.4 -> 74.9 mm, vias 0 -> 2
- net RX/TX: track 39.6 -> 40.9 mm
- net POWER_CHECK: track 52.7 -> 53.9 mm
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
Commit message: more datasheet
Routing:
- net RX/TX: track 40.9 -> 23.3 mm
- net CSN_nRF24: track 69.6 -> 60.1 mm

Commit message: V.2 controler
Parts:
- moved R5 0.41 mm to (137.2, 91.8)
- moved R6 0.41 mm to (136.6, 90.2)
Routing:
- net GND: track 47.4 -> 171.6 mm, vias 63 -> 24
- net SWDIO: track 37.2 -> 93.0 mm
- net L: track 76.5 -> 129.7 mm
- net SWDCK: track 37.7 -> 83.6 mm
- net Reset_Buton : track 32.7 -> 57.9 mm
- net Glob_Alim: track 258.2 -> 279.6 mm, vias 12 -> 7
- net RX/TX: track 23.3 -> 39.9 mm, vias 1 -> 2
- net Net-(D4-A): track 59.2 -> 73.6 mm, vias 0 -> 4
- net Net-(D8-A): track 14.6 -> 27.7 mm
- net Net-(D7-A): track 15.8 -> 28.8 mm
- net Net-(D9-A): track 13.8 -> 26.0 mm
- net R: track 74.9 -> 63.3 mm, vias 2 -> 4
- net DIODE_OE: track 59.0 -> 70.4 mm, vias 2 -> 3
- net Net-(D3-A): track 63.5 -> 74.3 mm, vias 0 -> 2
- net Order_Search: track 70.5 -> 81.2 mm
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Other:
- board text added: "B"
- board text added: "T"

Commit message: V.2.2
Routing:
- net GND: track 171.6 -> 191.2 mm, vias 24 -> 27
- net Glob_Alim: track 279.6 -> 275.9 mm

Commit message: change size vias
Routing:
- net GND: track 191.2 -> 82.2 mm, vias 27 -> 66
- net L: track 129.7 -> 118.4 mm
- net UC_Button: track 54.7 -> 57.6 mm
- net R: track 63.3 -> 65.9 mm, vias 4 -> 2
- net Net-(D4-A): track 74.1 -> 71.8 mm
- net A_Button: track 77.1 -> 74.9 mm
- net Net-(D5-A): track 59.7 -> 57.9 mm
- net Order_Search: track 81.2 -> 79.6 mm
- net NES/SNES_switcher: track 26.7 -> 28.0 mm
- net Y_Button: track 62.9 -> 61.7 mm
- net B_Button: track 74.6 -> 73.5 mm
- net Reset_Buton : track 57.9 -> 56.9 mm
- net Net-(D9-A): track 26.0 -> 25.3 mm
- net CSN_nRF24: track 51.5 -> 51.9 mm, vias 3 -> 2

Commit message: V.2.3
Connections:
- U1 pad 27: POWER_CHECK -> Order_Search
- U1 pad 7: Order_Search -> POWER_CHECK
Routing:
- net POWER_CHECK: track 54.6 -> 45.8 mm
- net Order_Search: track 79.6 -> 87.2 mm
Changed lines of the file:
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@@
   (net 83 "unconnected-(U5-P6-Pad19)")
   (net 84 "unconnected-(U5-P0-Pad10)")
-  (net 85 "Net-(U3-IN)")
+  (net 85 "Net-(FLG05-pwr)")
   (footprint "Resistor_SMD:R_0603_1608Metric_Pad0.98x0.95mm_HandSolder" (layer "F.Cu")
     (at 150.368 74.422)
@@
       (net 72 "unconnected-(U3-EN-Pad1)") (pinfunction "EN") (pintype "input+no_connect"))
     (pad "2" smd roundrect (at -2.1125 -0.325) (size 1.625 0.4) (layers "F.Cu" "F.Paste" "F.Mask") (roundrect_rratio 0.25)
-      (net 85 "Net-(U3-IN)") (pinfunction "IN") (pintype "power_in"))
+      (net 85 "Net-(FLG05-pwr)") (pinfunction "IN") (pintype "power_in"))
     (pad "3" smd roundrect (at -2.1125 0.325) (size 1.625 0.4) (layers "F.Cu" "F.Paste" "F.Mask") (roundrect_rratio 0.25)
       (net 5 "Glob_Alim") (pinfunction "OUT") (pintype "power_out"))
@@
       (net 3 "Li-ion") (pintype "passive"))
     (pad "2" smd rect (at 3.81 0 90) (size 1.6 0.76) (layers "F.Cu" "F.Paste" "F.Mask")
-      (net 85 "Net-(U3-IN)") (pintype "passive"))
+      (net 85 "Net-(FLG05-pwr)") (pintype "passive"))
     (model "${KICAD6_3DMODEL_DIR}/Button_Switch_SMD.3dshapes/SW_DIP_SPSTx01_Slide_Copal_CHS-01B_W7.62mm_P1.27mm.wrl"
       (offset (xyz 0 0 0))
@@
       (net 52 "B_Button") (pinfunction "PA0") (pintype "bidirectional"))
     (pad "7" smd roundrect (at -4.175 2 90) (size 1.5 0.5) (layers "F.Cu" "F.Paste" "F.Mask") (roundrect_rratio 0.25)
-      (net 65 "Order_Search") (pinfunction "PA1") (pintype "bidirectional"))
+      (net 1 "POWER_CHECK") (pinfunction "PA1") (pintype "bidirectional"))
     (pad "8" smd roundrect (at -4.175 2.8 90) (size 1.5 0.5) (layers "F.Cu" "F.Paste" "F.Mask") (roundrect_rratio 0.25)
       (net 48 "USART2_TX") (pinfunction "PA2") (pintype "bidirectional"))
@@
       (net 62 "DIODE_OE") (pinfunction "PB3") (pintype "bidirectional"))
     (pad "27" smd roundrect (at 1.2 -4.175 90) (size 0.5 1.5) (layers "F.Cu" "F.Paste" "F.Mask") (roundrect_rratio 0.25)
-      (net 1 "POWER_CHECK") (pinfunction "PB4") (pintype "bidirectional"))
+      (net 65 "Order_Search") (pinfunction "PB4") (pintype "bidirectional"))
     (pad "28" smd roundrect (at 0.4 -4.175 90) (size 0.5 1.5) (layers "F.Cu" "F.Paste" "F.Mask") (roundrect_rratio 0.25)
       (net 49 "NES{slash}SNES_switcher") (pinfunction "PB5") (pintype "bidirectional"))
@@
   )
   (segment (start 171.4 111.425) (end 173.35 111.425) (width 0.4) (layer "F.Cu") (net 1))
-  (segment (start 133.21 100.92) (end 133.24 100.95) (width 0.4) (layer "F.Cu") (net 1))
-  (segment (start 130.825 97.8) (end 131.588173 97.8) (width 0.4) (layer "F.Cu") (net 1))
+  (segment (start 137 107.42) (end 137.25 107.67) (width 0.4) (layer "F.Cu") (net 1))
   (segment (start 173.35 111.425) (end 173.4 111.475) (width 0.4) (layer "F.Cu") (net 1))
-  (segment (start 133.19 99.401827) (end 133.19 100.92) (width 0.4) (layer "F.Cu") (net 1))
-  (segment (start 133.19 100.92) (end 133.21 100.92) (width 0.4) (layer "F.Cu") (net 1))
+  (segment (start 137 103.175) (end 137 107.42) (width 0.4) (layer "F.Cu") (net 1))
   (segment (start 169.295 113.53) (end 171.4 111.425) (width 0.4) (layer "F.Cu") (net 1))
   (segment (start 173.4 111.475) (end 173.4 109.7125) (width 0.4) (layer "F.Cu") (net 1))
   (segment (start 168.8 113.53) (end 169.295 113.53) (width 0.4) (layer "F.Cu") (net 1))
-  (segment (start 131.588173 97.8) (end 133.19 99.401827) (width 0.4) (layer "F.Cu") (net 1))
+  (via (at 137.25 107.67) (size 1.6) (drill 0.8) (layers "F.Cu" "B.Cu") (net 1))
   (via (at 168.8 113.53) (size 1.6) (drill 0.8) (layers "F.Cu" "B.Cu") (net 1))
-  (via (at 133.24 100.95) (size 1.6) (drill 0.8) (layers "F.Cu" "B.Cu") (net 1))
   (segment (start 151.89 107.67) (end 157.75 113.53) (width 0.4) (layer "B.Cu") (net 1))
+  (segment (start 137.25 107.67) (end 151.89 107.67) (width 0.4) (layer "B.Cu") (net 1))
   (segment (start 157.75 113.53) (end 168.8 113.53) (width 0.4) (layer "B.Cu") (net 1))
-  (segment (start 136.59 107.67) (end 151.89 107.67) (width 0.4) (layer "B.Cu") (net 1))
-  (segment (start 133.24 104.32) (end 136.59 107.67) (width 0.4) (layer "B.Cu") (net 1))
-  (segment (start 133.24 100.95) (end 133.24 104.32) (width 0.4) (layer "B.Cu") (net 1))
   (segment (start 137.3 86.85) (end 137.05 87.1) (width 0.4) (layer "F.Cu") (net 2))
   (segment (start 138.35 87.8) (end 138.35 86.9) (width 0.4) (layer "F.Cu") (net 2))
@@
   (segment (start 140.803639 97) (end 140.932642 96.870998) (width 0.4) (layer "F.Cu") (net 64))
   (segment (start 139.175 97) (end 140.803639 97) (width 0.4) (layer "F.Cu") (net 64))
+  (segment (start 132.44 98.651827) (end 132.44 100.15) (width 0.4) (layer "F.Cu") (net 65))
+  (segment (start 132.44 100.15) (end 133.24 100.95) (width 0.4) (layer "F.Cu") (net 65))
+  (segment (start 130.825 97.8) (end 131.588173 97.8) (width 0.4) (layer "F.Cu") (net 65))
   (segment (start 180.489613 70.764613) (end 180.489613 70.8395) (width 0.4) (layer "F.Cu") (net 65))
   (segment (start 176.475 66.75) (end 180.489613 70.764613) (width 0.4) (layer "F.Cu") (net 65))
-  (segment (start 137 103.175) (end 137 106.08) (width 0.4) (layer "F.Cu") (net 65))
-  (segment (start 137 106.08) (end 137.32 106.4) (width 0.4) (layer "F.Cu") (net 65))
+  (segment (start 131.588173 97.8) (end 132.44 98.651827) (width 0.4) (layer "F.Cu") (net 65))
   (segment (start 176.475 66.75) (end 168.525 66.75) (width 0.4) (layer "F.Cu") (net 65))
-  (via (at 137.32 106.4) (size 1.6) (drill 0.8) (layers "F.Cu" "B.Cu") (net 65))
   (via (at 180.489613 70.8395) (size 1.6) (drill 0.8) (layers "F.Cu" "B.Cu") (net 65))
-  (segment (start 137.32 106.4) (end 149.82 106.4) (width 0.4) (layer "B.Cu") (net 65))
+  (via (at 133.24 100.95) (size 1.6) (drill 0.8) (layers "F.Cu" "B.Cu") (net 65))
+  (segment (start 162.92 91.98) (end 166.55 88.35) (width 0.4) (layer "B.Cu") (net 65))
+  (segment (start 138.69 106.4) (end 149.82 106.4) (width 0.4) (layer "B.Cu") (net 65))
   (segment (start 170.8 80.529113) (end 180.489613 70.8395) (width 0.4) (layer "B.Cu") (net 65))
+  (segment (start 162.92 93.3) (end 162.92 91.98) (width 0.4) (layer "B.Cu") (net 65))
   (segment (start 149.82 106.4) (end 162.92 93.3) (width 0.4) (layer "B.Cu") (net 65))
-  (segment (start 162.92 91.98) (end 166.55 88.35) (width 0.4) (layer "B.Cu") (net 65))
-  (segment (start 166.55 88.35) (end 169.65 88.35) (width 0.4) (layer "B.Cu") (net 65))
   (segment (start 169.65 88.35) (end 170.8 87.2) (width 0.4) (layer "B.Cu") (net 65))
-  (segment (start 162.92 93.3) (end 162.92 91.98) (width 0.4) (layer "B.Cu") (net 65))
   (segment (start 170.8 87.2) (end 170.8 80.529113) (width 0.4) (layer "B.Cu") (net 65))
+  (segment (start 166.55 88.35) (end 169.65 88.35) (width 0.4) (layer "B.Cu") (net 65))
+  (segment (start 133.24 100.95) (end 138.69 106.4) (width 0.4) (layer "B.Cu") (net 65))
   (segment (start 136.7805 67.4895) (end 136.7805 79.077727) (width 0.4) (layer "F.Cu") (net 66))
   (segment (start 142.2 64.6) (end 139.67 64.6) (width 0.4) (layer "F.Cu") (net 66))

Commit message: V.2.4
Parts:
- C1: value 100uF -> 22uF; footprint Capacitor_SMD:C_0603_1608Metric_Pad1.08x0.95mm_HandSolder -> Capacitor_SMD:CP_Elec_5x5.4
- moved C1 2.32 mm to (137.4, 64.0)
Routing:
- net GND: track 82.2 -> 94.8 mm, vias 66 -> 67
- net Net-(D6-A): track 50.4 -> 49.2 mm
- net CSN_nRF24: track 51.9 -> 50.7 mm
- net MOSI: track 42.7 -> 43.7 mm
