File: Hardware/Kicad/Controler_NRF24L01_Exclude_v3/Controler_NRF24L01_Exclude_v3.kicad_pcb (KiCad board)
At the start: 2 copper layers, 160.2 x 60.2 mm, 87 parts, among them J1 Conn_01x02, J2 Conn_02x07_Odd_Even, J3 Conn_01x03, J4 Conn_01x03, SW1 SW_DIP_x01, SW10 SW_DIP_x01, SW11 SW_Push, SW12 SW_Push, SW13 SW_Push, SW2 SW_Push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

Commit message: Controler V.3 and Shell rebuild
Parts:
- moved C4 10.7 mm to (169.8, 85.5)
- moved SW1 10.6 mm to (168.9, 79.9)
Routing:
- net Li-ion: track 26.0 -> 36.6 mm
- net Net-(#FLG05-pwr): track 15.4 -> 7.92 mm
- net GND: track 62.9 -> 70.2 mm
- net Net-(D10-A): track 23.0 -> 29.6 mm
- net Net-(D18-A): track 6.45 -> 7.03 mm
Changed lines of the file:
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@@
   )
   (footprint "Capacitor_SMD:C_0603_1608Metric_Pad1.08x0.95mm_HandSolder" (layer "F.Cu")
-    (at 169.785 96.17)
+    (at 169.785 85.5)
     (descr "Capacitor SMD 0603 (1608 Metric), square (rectangular) end terminal, IPC_7351 nominal with elongated pad for handsoldering. (Body size source: IPC-SM-782 page 76, https://www.pcb-3d.com/wordpress/wp-content/uploads/ipc-sm-782a_amendment_1_and_2.pdf), generated with kicad-footprint-generator")
     (tags "capacitor handsolder")
@@
   )
   (footprint "Button_Switch_SMD:SW_DIP_SPSTx01_Slide_Copal_CHS-01B_W7.62mm_P1.27mm" (layer "F.Cu")
-    (at 168.86 90.47 90)
+    (at 168.86 79.9 90)
     (descr "SMD 1x-dip-switch SPST Copal_CHS-01B, Slide, row spacing 7.62 mm (300 mils), body size  (see http://www.nidec-copal-electronics.com/e/catalog/switch/chs.pdf), SMD")
     (tags "SMD DIP Switch SPST Slide 7.62mm 300mil SMD")
@@
   (segment (start 146.36 78.94) (end 147.61 77.69) (width 0.4) (layer "F.Cu") (net 2))
   (segment (start 159.149 79.55) (end 159.149 81.6765) (width 0.4) (layer "F.Cu") (net 2))
+  (segment (start 160.049 80.45) (end 165.75 80.45) (width 0.4) (layer "F.Cu") (net 2))
   (segment (start 148.89 98.45) (end 148.89 93.05) (width 0.4) (layer "F.Cu") (net 2))
   (segment (start 159.149 75.9515) (end 159.799 75.9515) (width 0.4) (layer "F.Cu") (net 2))
@@
   (segment (start 159.149 79.511183) (end 157.849 80.811183) (width 0.4) (layer "F.Cu") (net 2))
   (segment (start 144.914 99.2345) (end 145.2145 99.2345) (width 0.4) (layer "F.Cu") (net 2))
+  (segment (start 167.76 74.61) (end 168.25 74.12) (width 0.4) (layer "F.Cu") (net 2))
+  (segment (start 168.25 74.12) (end 172.03 74.12) (width 0.4) (layer "F.Cu") (net 2))
   (segment (start 146.36 82.33) (end 146.36 78.94) (width 0.4) (layer "F.Cu") (net 2))
   (segment (start 147.17 100.17) (end 148.89 98.45) (width 0.4) (layer "F.Cu") (net 2))
   (segment (start 145.2145 99.2345) (end 146.15 100.17) (width 0.4) (layer "F.Cu") (net 2))
+  (segment (start 165.75 80.45) (end 167.76 78.44) (width 0.4) (layer "F.Cu") (net 2))
   (segment (start 159.149 79.55) (end 157.59 79.55) (width 0.4) (layer "F.Cu") (net 2))
+  (segment (start 165.75 80.45) (end 166.24 80.45) (width 0.4) (layer "F.Cu") (net 2))
   (segment (start 157.59 79.55) (end 157.28 79.86) (width 0.4) (layer "F.Cu") (net 2))
   (segment (start 166.24 80.45) (end 166.24 81.0855) (width 0.4) (layer "F.Cu") (net 2))
   (segment (start 144.914 99.2345) (end 143.39 99.2345) (width 0.4) (layer "F.Cu") (net 2))
   (segment (start 159.149 79.511183) (end 159.149 79.55) (width 0.4) (layer "F.Cu") (net 2))
-  (segment (start 166.24 80.45) (end 168.98 77.71) (width 0.4) (layer "F.Cu") (net 2))
-  (segment (start 160.049 80.45) (end 166.24 80.45) (width 0.4) (layer "F.Cu") (net 2))
+  (segment (start 167.76 78.44) (end 167.76 74.61) (width 0.4) (layer "F.Cu") (net 2))
   (segment (start 157.849 80.811183) (end 157.849 81.6765) (width 0.4) (layer "F.Cu") (net 2))
   (segment (start 159.149 75.9515) (end 159.149 79.511183) (width 0.4) (layer "F.Cu") (net 2))
   (via (at 153.67 82.14) (size 1.6) (drill 0.8) (layers "F.Cu" "B.Cu") (free) (net 2))
-  (via (at 168.98 77.71) (size 1.6) (drill 0.8) (layers "F.Cu" "B.Cu") (free) (net 2))
+  (via (at 172.03 74.12) (size 1.6) (drill 0.8) (layers "F.Cu" "B.Cu") (free) (net 2))
   (via (at 148.89 93.05) (size 1.6) (drill 0.8) (layers "F.Cu" "B.Cu") (free) (net 2))
   (via (at 147.61 77.69) (size 1.6) (drill 0.8) (layers "F.Cu" "B.Cu") (net 2))
@@
   (segment (start 140.69 108.075) (end 140.69 115.44) (width 0.4) (layer "F.Cu") (net 3))
   (segment (start 177.09 112.7875) (end 180.4525 112.7875) (width 0.4) (layer "F.Cu") (net 4))
-  (segment (start 169.71 96.9575) (end 168.9225 96.17) (width 0.4) (layer "F.Cu") (net 4))
+  (segment (start 168.86 83.71) (end 168.86 85.4375) (width 0.4) (layer "F.Cu") (net 4))
+  (segment (start 169.71 86.2875) (end 168.9225 85.5) (width 0.4) (layer "F.Cu") (net 4))
   (segment (start 169.71 105.4075) (end 169.71 96.9575) (width 0.4) (layer "F.Cu") (net 4))
-  (segment (start 168.9225 94.3425) (end 168.86 94.28) (width 0.4) (layer "F.Cu") (net 4))
-  (segment (start 168.9225 96.17) (end 168.9225 94.3425) (width 0.4) (layer "F.Cu") (net 4))
+  (segment (start 169.71 96.9575) (end 169.71 86.2875) (width 0.4) (layer "F.Cu") (net 4))
+  (segment (start 168.86 85.4375) (end 168.9225 85.5) (width 0.4) (layer "F.Cu") (net 4))
   (segment (start 177.09 112.7875) (end 169.71 105.4075) (width 0.4) (layer "F.Cu") (net 4))
   (segment (start 180.4525 112.7875) (end 180.965 113.3) (width 0.4) (layer "F.Cu") (net 4))
@@
   (segment (start 157.59 69.675) (end 157.415 69.85) (width 0.5) (layer "F.Cu") (net 23))
   (segment (start 157.59 68.125) (end 157.59 69.675) (width 0.5) (layer "F.Cu") (net 23))
-  (segment (start 166.717183 84.26) (end 166.78 84.26) (width 0.4) (layer "F.Cu") (net 24))
   (segment (start 157.415 73.695) (end 157.45 73.73) (width 0.4) (layer "F.Cu") (net 24))
-  (segment (start 164.999 82.541817) (end 166.717183 84.26) (width 0.4) (layer "F.Cu") (net 24))
+  (segment (start 164.999 82.541817) (end 166.5 84.042817) (width 0.4) (layer "F.Cu") (net 24))
   (segment (start 157.415 71.6) (end 157.415 73.695) (width 0.4) (layer "F.Cu") (net 24))
+  (segment (start 166.5 84.042817) (end 166.5 87.94) (width 0.4) (layer "F.Cu") (net 24))
   (segment (start 164.999 81.6765) (end 164.999 82.541817) (width 0.4) (layer "F.Cu") (net 24))
-  (via (at 166.78 84.26) (size 1.6) (drill 0.8) (layers "F.Cu" "B.Cu") (net 24))
+  (via (at 166.5 87.94) (size 1.6) (drill 0.8) (layers "F.Cu" "B.Cu") (net 24))
   (via (at 157.45 73.73) (size 1.6) (drill 0.8) (layers "F.Cu" "B.Cu") (net 24))
-  (segment (start 157.45 74.46) (end 157.89 74.9) (width 0.4) (layer "B.Cu") (net 24))
-  (segment (start 157.45 73.73) (end 157.45 74.46) (width 0.4) (layer "B.Cu") (net 24))
-  (segment (start 166.74 78.53) (end 166.74 84.22) (width 0.4) (layer "B.Cu") (net 24))
-  (segment (start 166.74 84.22) (end 166.78 84.26) (width 0.4) (layer "B.Cu") (net 24))
-  (segment (start 157.89 74.9) (end 163.11 74.9) (width 0.4) (layer "B.Cu") (net 24))
-  (segment (start 163.11 74.9) (end 166.74 78.53) (width 0.4) (layer "B.Cu") (net 24))
+  (segment (start 166.5 78.29) (end 166.5 87.94) (width 0.4) (layer "B.Cu") (net 24))
+  (segment (start 157.45 73.73) (end 161.94 73.73) (width 0.4) (layer "B.Cu") (net 24))
+  (segment (start 161.94 73.73) (end 166.5 78.29) (width 0.4) (layer "B.Cu") (net 24))
   (segment (start 159.09 68.125) (end 159.09 69.775) (width 0.5) (layer "F.Cu") (net 25))
   (segment (start 159.09 69.775) (end 159.015 69.85) (width 0.5) (layer "F.Cu") (net 25))
@@
   (segment (start 169.59 69.125) (end 170.29 69.825) (width 0.5) (layer "F.Cu") (net 39))
   (segment (start 169.59 68.125) (end 169.59 69.125) (width 0.5) (layer "F.Cu") (net 39))
-  (segment (start 165.9135 75.9515) (end 170.29 71.575) (width 0.4) (layer "F.Cu") (net 40))
-  (segment (start 165.649 75.9515) (end 165.9135 75.9515) (width 0.4) (layer "F.Cu") (net 40))
+  (segment (start 168.551466 72.9) (end 169.8 72.9) (width 0.4) (layer "F.Cu") (net 40))
+  (segment (start 165.649 75.802466) (end 168.551466 72.9) (width 0.4) (layer "F.Cu") (net 40))
+  (segment (start 170.29 72.41) (end 170.29 71.575) (width 0.4) (layer "F.Cu") (net 40))
+  (segment (start 169.8 72.9) (end 170.29 72.41) (width 0.4) (layer "F.Cu") (net 40))
+  (segment (start 165.649 75.9515) (end 165.649 75.802466) (width 0.4) (layer "F.Cu") (net 40))
   (segment (start 167.55 107.95) (end 164.2 111.3) (width 0.4) (layer "F.Cu") (net 43))
   (segment (start 136.69 99.725) (end 136.69 103.02) (width 0.4) (layer "F.Cu") (net 43))
@@
   (segment (start 142.673428 79.246572) (end 153.836246 79.246572) (width 0.4) (layer "B.Cu") (net 56))
   (segment (start 161.13 78.51) (end 154.572818 78.51) (width 0.4) (layer "B.Cu") (net 56))
-  (segment (start 172.945 76.575) (end 176.5775 76.575) (width 0.4) (layer "F.Cu") (net 57))
-  (segment (start 168.86 80.66) (end 172.945 76.575) (width 0.4) (layer "F.Cu") (net 57))
-  (segment (start 168.86 86.66) (end 168.86 80.66) (width 0.4) (layer "F.Cu") (net 57))
+  (segment (start 169.345 76.575) (end 168.86 76.09) (width 0.4) (layer "F.Cu") (net 57))
+  (segment (start 176.5775 76.575) (end 169.345 76.575) (width 0.4) (layer "F.Cu") (net 57))
   (segment (start 211.665 94.15) (end 203.715 94.15) (width 0.4) (layer "F.Cu") (net 58))
   (segment (start 203.715 94.15) (end 201.21 91.645) (width 0.4) (layer "F.Cu") (net 58))

Commit message: final version
Parts:
- moved C4 0.10 mm to (169.8, 85.6)
Routing:
- net GND: track 70.2 -> 100.6 mm, vias 6 -> 9
- net Net-(D3-A): track 84.2 -> 85.8 mm
- net Net-(C8-Pad1): track 0.00 -> 1.62 mm
- net Net-(D4-A): track 77.7 -> 79.3 mm
- net A_Button: track 23.0 -> 21.9 mm
Changed lines of the file:
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@@
   )
   (footprint "Capacitor_SMD:C_0603_1608Metric_Pad1.08x0.95mm_HandSolder" (layer "F.Cu")
-    (at 169.785 85.5)
+    (at 169.785 85.6)
     (descr "Capacitor SMD 0603 (1608 Metric), square (rectangular) end terminal, IPC_7351 nominal with elongated pad for handsoldering. (Body size source: IPC-SM-782 page 76, https://www.pcb-3d.com/wordpress/wp-content/uploads/ipc-sm-782a_amendment_1_and_2.pdf), generated with kicad-footprint-generator")
     (tags "capacitor handsolder")
@@
   (via (at 148.89 93.05) (size 1.6) (drill 0.8) (layers "F.Cu" "B.Cu") (free) (net 2))
   (via (at 147.61 77.69) (size 1.6) (drill 0.8) (layers "F.Cu" "B.Cu") (net 2))
+  (via (at 117.9 71.25) (size 1.6) (drill 0.8) (layers "F.Cu" "B.Cu") (free) (net 2))
   (via (at 146.36 82.33) (size 1.6) (drill 0.8) (layers "F.Cu" "B.Cu") (free) (net 2))
+  (via (at 123.07 70.94) (size 1.6) (drill 0.8) (layers "F.Cu" "B.Cu") (free) (net 2))
+  (via (at 114.35 71.34) (size 1.6) (drill 0.8) (layers "F.Cu" "B.Cu") (free) (net 2))
   (via (at 157.28 79.86) (size 1.6) (drill 0.8) (layers "F.Cu" "B.Cu") (net 2))
+  (segment (start 198.925 92.055) (end 199.03 91.95) (width 0.4) (layer "B.Cu") (net 2))
+  (segment (start 202.07 89.1) (end 202.07 91.45) (width 0.4) (layer "B.Cu") (net 2))
+  (segment (start 114.44 71.25) (end 114.35 71.34) (width 0.4) (layer "B.Cu") (net 2))
+  (segment (start 199.03 91.95) (end 195.12 91.95) (width 0.4) (layer "B.Cu") (net 2))
   (segment (start 157.28 79.86) (end 155.95 79.86) (width 0.4) (layer "B.Cu") (net 2))
+  (segment (start 195.675 88) (end 195.725 88.05) (width 0.4) (layer "B.Cu") (net 2))
   (segment (start 95.925 92.065) (end 95.925 92.9) (width 0.4) (layer "B.Cu") (net 2))
+  (segment (start 193.775 91.95) (end 193.725 92) (width 0.4) (layer "B.Cu") (net 2))
+  (segment (start 195.725 88.05) (end 201.02 88.05) (width 0.4) (layer "B.Cu") (net 2))
+  (segment (start 195.675 87.1) (end 195.675 88) (width 0.4) (layer "B.Cu") (net 2))
   (segment (start 90.725 92.9) (end 90.725 90) (width 0.4) (layer "B.Cu") (net 2))
+  (segment (start 202.07 91.45) (end 201.57 91.95) (width 0.4) (layer "B.Cu") (net 2))
+  (segment (start 198.925 92.9) (end 198.925 92.055) (width 0.4) (layer "B.Cu") (net 2))
+  (segment (start 195.025 92.045) (end 195.12 91.95) (width 0.4) (layer "B.Cu") (net 2))
+  (segment (start 195.12 91.95) (end 193.775 91.95) (width 0.4) (layer "B.Cu") (net 2))
+  (segment (start 201.02 88.05) (end 202.07 89.1) (width 0.4) (layer "B.Cu") (net 2))
+  (segment (start 117.9 71.25) (end 122.76 71.25) (width 0.4) (layer "B.Cu") (net 2))
   (segment (start 92.675 88.815) (end 95.925 92.065) (width 0.4) (layer "B.Cu") (net 2))
   (segment (start 92.675 92.9) (end 92.675 88.05) (width 0.4) (layer "B.Cu") (net 2))
@@
   (segment (start 92.675 88.05) (end 92.675 88.815) (width 0.4) (layer "B.Cu") (net 2))
   (segment (start 155.95 79.86) (end 153.67 82.14) (width 0.4) (layer "B.Cu") (net 2))
+  (segment (start 117.9 71.25) (end 114.44 71.25) (width 0.4) (layer "B.Cu") (net 2))
+  (segment (start 195.025 92.9) (end 195.025 92.045) (width 0.4) (layer "B.Cu") (net 2))
+  (segment (start 201.57 91.95) (end 199.03 91.95) (width 0.4) (layer "B.Cu") (net 2))
   (segment (start 90.725 90) (end 92.675 88.05) (width 0.4) (layer "B.Cu") (net 2))
+  (segment (start 122.76 71.25) (end 123.07 70.94) (width 0.4) (layer "B.Cu") (net 2))
+  (segment (start 193.725 92) (end 193.725 92.9) (width 0.4) (layer "B.Cu") (net 2))
   (segment (start 177.04 116.325) (end 177.09 116.375) (width 0.4) (layer "F.Cu") (net 3))
   (segment (start 170.075 121.34) (end 175.09 116.325) (width 0.4) (layer "F.Cu") (net 3))
@@
   (segment (start 180.4525 112.7875) (end 180.965 113.3) (width 0.4) (layer "F.Cu") (net 4))
   (segment (start 203.589524 98.45) (end 201.864524 98.45) (width 0.4) (layer "F.Cu") (net 5))
+  (segment (start 89.735476 98.45) (end 88.110476 98.45) (width 0.4) (layer "F.Cu") (net 6))
   (segment (start 175.515 78.9375) (end 176.5775 77.875) (width 0.4) (layer "F.Cu") (net 7))
   (segment (start 174.74 78.9375) (end 175.515 78.9375) (width 0.4) (layer "F.Cu") (net 7))
@@
   (segment (start 110.715 67.4625) (end 110.715 66) (width 0.4) (layer "F.Cu") (net 9))
   (segment (start 110.715 66) (end 110.815 65.9) (width 0.4) (layer "F.Cu") (net 9))
-  (segment (start 112.565 69.285) (end 112.565 65.9) (width 0.4) (layer "F.Cu") (net 10))
-  (segment (start 134.985 91.705) (end 134.985 80.825) (width 0.4) (layer "F.Cu") (net 10))
-  (segment (start 128.65 74.49) (end 117.8 74.49) (width 0.4) (layer "F.Cu") (net 10))
+  (segment (start 134.985 80.825) (end 134.985 91.705) (width 0.4) (layer "F.Cu") (net 10))
+  (segment (start 112.565 65.9) (end 112.565 72.085) (width 0.4) (layer "F.Cu") (net 10))
   (segment (start 162.399 83.971) (end 162.399 81.6765) (width 0.4) (layer "F.Cu") (net 10))
-  (segment (start 134.985 80.825) (end 128.65 74.49) (width 0.4) (layer "F.Cu") (net 10))
+  (segment (start 114.97 74.49) (end 128.65 74.49) (width 0.4) (layer "F.Cu") (net 10))
+  (segment (start 134.985 91.705) (end 136.42 93.14) (width 0.4) (layer "F.Cu") (net 10))
   (segment (start 161.04 85.33) (end 162.399 83.971) (width 0.4) (layer "F.Cu") (net 10))
   (segment (start 162.07 88.29) (end 162.07 87.52) (width 0.4) (layer "F.Cu") (net 10))
-  (segment (start 117.785 74.505) (end 112.565 69.285) (width 0.4) (layer "F.Cu") (net 10))
-  (segment (start 136.42 94.41) (end 136.42 93.14) (width 0.4) (layer "F.Cu") (net 10))
-  (segment (start 136.42 93.14) (end 134.985 91.705) (width 0.4) (layer "F.Cu") (net 10))
   (segment (start 161.04 86.49) (end 161.04 85.33) (width 0.4) (layer "F.Cu") (net 10))
   (segment (start 162.07 87.52) (end 161.04 86.49) (width 0.4) (layer "F.Cu") (net 10))
-  (segment (start 117.8 74.49) (end 117.785 74.505) (width 0.4) (layer "F.Cu") (net 10))
+  (segment (start 112.565 72.085) (end 114.97 74.49) (width 0.4) (layer "F.Cu") (net 10))
+  (segment (start 136.42 93.14) (end 136.42 94.41) (width 0.4) (layer "F.Cu") (net 10))
+  (segment (start 128.65 74.49) (end 134.985 80.825) (width 0.4) (layer "F.Cu") (net 10))
   (via (at 136.42 94.41) (size 1.6) (drill 0.8) (layers "F.Cu" "B.Cu") (net 10))
   (via (at 162.07 88.29) (size 1.6) (drill 0.8) (layers "F.Cu" "B.Cu") (net 10))
@@
   (segment (start 114.215 67.4875) (end 114.215 66) (width 0.4) (layer "F.Cu") (net 11))
   (segment (start 114.215 66) (end 114.315 65.9) (width 0.4) (layer "F.Cu") (net 11))
-  (segment (start 129.44 73.65) (end 120.27 73.65) (width 0.4) (layer "F.Cu") (net 12))
+  (segment (start 116.065 72.185) (end 117.53 73.65) (width 0.4) (layer "F.Cu") (net 12))
+  (segment (start 136.01 80.22) (end 136.01 91.45) (width 0.4) (layer "F.Cu") (net 12))
   (segment (start 160.08 85.17) (end 161.749 83.501) (width 0.4) (layer "F.Cu") (net 12))
   (segment (start 161.749 83.501) (end 161.749 81.6765) (width 0.4) (layer "F.Cu") (net 12))
-  (segment (start 136.01 80.22) (end 129.44 73.65) (width 0.4) (layer "F.Cu") (net 12))
-  (segment (start 138.08 93.52) (end 136.01 91.45) (width 0.4) (layer "F.Cu") (net 12))
-  (segment (start 120.27 73.65) (end 116.065 69.445) (width 0.4) (layer "F.Cu") (net 12))
+  (segment (start 116.065 65.9) (end 116.065 72.185) (width 0.4) (layer "F.Cu") (net 12))
+  (segment (start 117.53 73.65) (end 129.44 73.65) (width 0.4) (layer "F.Cu") (net 12))
+  (segment (start 136.01 91.45) (end 138.08 93.52) (width 0.4) (layer "F.Cu") (net 12))
+  (segment (start 129.44 73.65) (end 136.01 80.22) (width 0.4) (layer "F.Cu") (net 12))
   (segment (start 160.08 89.31) (end 160.08 85.17) (width 0.4) (layer "F.Cu") (net 12))
-  (segment (start 136.01 91.45) (end 136.01 80.22) (width 0.4) (layer "F.Cu") (net 12))
-  (segment (start 116.065 69.445) (end 116.065 65.9) (width 0.4) (layer "F.Cu") (net 12))
   (via (at 138.08 93.52) (size 1.6) (drill 0.8) (layers "F.Cu" "B.Cu") (net 12))
   (via (at 160.08 89.31) (size 1.6) (drill 0.8) (layers "F.Cu" "B.Cu") (net 12))
@@
   (segment (start 169.345 76.575) (end 168.86 76.09) (width 0.4) (layer "F.Cu") (net 57))
   (segment (start 176.5775 76.575) (end 169.345 76.575) (width 0.4) (layer "F.Cu") (net 57))
+  (segment (start 203.59 94.15) (end 200.65 91.21) (width 0.4) (layer "F.Cu") (net 58))
   (segment (start 211.665 94.15) (end 203.715 94.15) (width 0.4) (layer "F.Cu") (net 58))
-  (segment (start 203.715 94.15) (end 201.21 91.645) (width 0.4) (layer "F.Cu") (net 58))
-  (segment (start 201.21 91.645) (end 201.21 88.9) (width 0.4) (layer "F.Cu") (net 58))
-  (via (at 201.21 88.9) (size 1.6) (drill 0.8) (layers "F.Cu" "B.Cu") (net 58))
-  (segment (start 194.575 88.9) (end 201.21 88.9) (width 0.4) (layer "B.Cu") (net 58))
-  (segment (start 193.725 88.05) (end 194.575 88.9) (width 0.4) (layer "B.Cu") (net 58))
+  (segment (start 203.715 94.15) (end 203.59 94.15) (width 0.4) (layer "F.Cu") (net 58))
+  (segment (start 200.65 91.21) (end 200.65 90.33) (width 0.4) (layer "F.Cu") (net 58))
+  (via (at 200.65 90.33) (size 1.6) (drill 0.8) (layers "F.Cu" "B.Cu") (net 58))
   (segment (start 193.725 87.1) (end 193.725 88.05) (width 0.4) (layer "B.Cu") (net 58))
+  (segment (start 193.725 88.05) (end 196.005 90.33) (width 0.4) (layer "B.Cu") (net 58))
+  (segment (start 196.005 90.33) (end 200.65 90.33) (width 0.4) (layer "B.Cu") (net 58))
   (segment (start 191.36 96.81) (end 191.36 91.61) (width 0.4) (layer "F.Cu") (net 59))
   (segment (start 191.36 91.61) (end 186.04 86.29) (width 0.4) (layer "F.Cu") (net 59))

Commit message: fix pcb v3
Routing:
- net GND: track 100.6 -> 115.5 mm, vias 9 -> 14
- net Pin_Clock: track 52.3 -> 57.3 mm
- net Digital_Out_Put: track 44.3 -> 49.0 mm
- net MOSI: track 45.3 -> 49.3 mm
- net Reset_Buton : track 52.9 -> 49.0 mm
- net Glob_Alim: track 391.7 -> 395.4 mm
- net DIO/EX_CLK: track 187.7 -> 186.1 mm
- net DIO/EX_SDA: track 172.2 -> 170.7 mm
- net R: track 28.7 -> 29.8 mm
Other:
- board size 160.2 x 60.2 mm -> 157.5 x 58 mm
